File: boneIO - input WT32.kicad_sch (KiCad schematic)
At the start: 347 parts, among them J1 POWER, J10 P5, J11 P6, J12 P7, J2 GT-USB-7010AN, J3 UART, J4 EXT_PSU, J5 Conn_02x04_Odd_Even, J6 P1, J7 P2, J8 P4, J9 P3, Q1 AO3401A, Q2 SS8050, Q3 SS8050, SW1 SW_DIP_x04, SW2 USER_SWITCH, U1 SN65HVD230, U10 EL357N, U11 EL357N, U12 EL357N, U13 EL357N, U14 EL357N, U15 EL357N, U16 RS485, U17 XL1509-5, U18 USBLC6-2SC6, U19 CH340C, U2 WT32-ETH01, U20 EL357N, U21 EL357N, U22 EL357N, U23 EL357N, U24 EL357N, U25 EL357N, U26 RT9013-33GB, U27 LM358, U28 EL357N, U29 EL357N, U3 EL357N, U30 EL357N, U31 EL357N, U32 EL357N, U33 EL357N, U34 2N7002DW/BSS138PS, U35 DS1307Z+, U36 EL357N, U37 EL357N, U38 EL357N, U39 EL357N, U4 EL357N, U40 EL357N, U41 EL357N, U42 PCA9515, U43 PCA9515, U44 EL357N, U45 EL357N, U46 EL357N, U47 EL357N, U48 EL357N, U49 MCP23017_SS, U5 EL357N, U50 PCF8575, U51 SN74LVC1G3157, U52 PCF8575, U53 MCP23017_SS, U54 SN74LVC1G3157, U6 EL357N, U7 EL357N, U8 EL357N, U9 INA219AxD, Y1 32,788 MHz

Commit message: input_board_ESP_v0.4
Project changes:
- improving GND polygons
- improving the power supply circuit from USB
Parts:
- removed R54: 0k, Resistor_SMD:R_0603_1608Metric, symbol Device:R
- removed U18: USBLC6-2SC6, Package_TO_SOT_SMD:SOT-23-6, symbol Power_Protection:USBLC6-2SC6
- added A1: Opened, Jumper:SolderJumper-2_P1.3mm_Open_RoundedPad1.0x1.5mm, symbol ESP32-EVB_Rev_I:SJ
- added C35, C36, C37: 100n, Capacitor_SMD:C_0603_1608Metric, symbol Device:C
- added D32: 1N4148, Diode_SMD:D_MiniMELF, symbol Device:D
- added D33: SMBJ5.0A, Diode_SMD:D_SMB, symbol Diode:SM6T18A
- added D34: SM712_SOT23, Package_TO_SOT_SMD:SOT-23, symbol Diode:SM712_SOT23
- added F3: 6V 500mA, Fuse:Fuse_1206_3216Metric, symbol Device:Fuse
- added R70, R87, R94, R95: 4.7k, Resistor_SMD:R_0603_1608Metric, symbol Device:R
- added R84: 56k, Resistor_SMD:R_0603_1608Metric, symbol Device:R
- added R96: 120R, Resistor_SMD:R_0805_2012Metric, symbol Device:R
- added U25: 74HC14, Package_SO:SO-14_3.9x8.65mm_P1.27mm, symbol 74xx:74HC14
- added U33: MAX485E, Package_SO:SO-8_3.9x4.9mm_P1.27mm, symbol Interface_UART:MAX485E
- renumbered A1 to A5, A5 to A6, A6 to A7, A7 to A8, C2 to C1, C12 to C10, C13 to C11, C14 to C12, C15 to C13, C16 to C14, C17 to C15, C19 to C16, C11 to C17, C21 to C18, C22 to C19, C3 to C2, C23 to C20, C24 to C21, C25 to C22, C26 to C23, C27 to C24, C29 to C25, C30 to C26, C31 to C27, C32 to C28, C33 to C29, C4 to C3, C34 to C30, C35 to C31, C36 to C32, C37 to C33, C10 to C34, C40 to C38, C41 to C39, C5 to C4, C42 to C40, C43 to C41, C44 to C42, C45 to C43, C20 to C44, C28 to C45, C48 to C46, C49 to C47, C50 to C48, C51 to C49, C6 to C5, C52 to C50, C38 to C51, C39 to C52, C1 to C53, C53 to C54, C47 to C55, C46 to C56, C54 to C57, C7 to C6, C8 to C7, C18 to C8, D17 to D10, D18 to D17, D19 to D18, D20 to D19, D21 to D20, D22 to D21, D23 to D22, D24 to D23, D25 to D24, D26 to D25, D29 to D26, D30 to D27, D31 to D28, D32 to D29, D4 to D3, D33 to D30, D34 to D31, D37 to D35, D38 to D36, D39 to D37, D40 to D38, D41 to D39, D5 to D4, D42 to D40, D27 to D41, D28 to D42, D45 to D43, D46 to D44, D47 to D45, D48 to D46, D49 to D47, D43 to D48, D3 to D49, D6 to D5, D35 to D50, D36 to D51, D44 to D52, D7 to D6, D8 to D7, D9 to D8, D10 to D9, J11 to J10, J12 to J11, J4 to J12, J6 to J4, J7 to J5, J5 to J6, J8 to J7, J9 to J8, J10 to J9, R2 to R1, R13 to R10, R111 to R100, R112 to R101, R113 to R102, R114 to R103, R115 to R104, R116 to R105, R117 to R106, R118 to R107, R119 to R108, R69 to R109, R14 to R11, R70 to R110, R122 to R111, R123 to R112, R124 to R113, R125 to R114, R126 to R115, R68 to R116, R73 to R117, R74 to R118, R71 to R119, R15 to R12, R128 to R120, R129 to R121, R130 to R122, R131 to R123, R132 to R124, R133 to R125, R82 to R126, R135 to R127, R136 to R128, R137 to R129, R17 to R13, R138 to R130, R83 to R131, R96 to R132, R97 to R133, R98 to R134, R99 to R135, R106 to R136, R107 to R137, R1 to R138, R18 to R14, R8 to R143, R9 to R144, R120 to R145, R16 to R146, R121 to R147, R143 to R148, R145 to R149, R19 to R15, R146 to R150, R147 to R151, R127 to R152, R134 to R153, R20 to R16, R21 to R17, R22 to R18, R25 to R19, R3 to R2, R23 to R20, R24 to R21, R26 to R22, R27 to R23, R28 to R24, R29 to R25, R30 to R26, R31 to R27, R47 to R28, R34 to R29, R4 to R3, R35 to R30, R36 to R31, R37 to R32, R38 to R33, R39 to R34, R41 to R35, R42 to R36, R43 to R37, R44 to R38, R45 to R39, R5 to R4, R46 to R40, R55 to R41, R48 to R42, R49 to R43, R50 to R44, R51 to R45, R52 to R46, R53 to R47, R144 to R48, R72 to R49, R6 to R5, R56 to R50, R57 to R51, R58 to R52, R59 to R53, R60 to R54, R61 to R55, R62 to R56, R63 to R57, R64 to R58, R65 to R59, R7 to R6, R66 to R60, R67 to R61, R81 to R62, R148 to R63, R75 to R64, R76 to R65, R77 to R66, R78 to R67, R79 to R68, R80 to R69, R10 to R7, R32 to R71, R84 to R72, R85 to R73, R86 to R74, R87 to R75, R88 to R76, R89 to R77, R90 to R78, R91 to R79, R11 to R8, R92 to R80, R93 to R81, R94 to R82, R95 to R83, R33 to R85, R40 to R86, R100 to R88, R101 to R89, R12 to R9, R102 to R90, R103 to R91, R104 to R92, R105 to R93, R108 to R97, R109 to R98, R110 to R99, SW2 to SW1, SW1 to SW2, U3 to U1, U11 to U10, U12 to U11, U13 to U12, U14 to U13, U15 to U14, U17 to U15, U20 to U17, U21 to U18, U22 to U19, U4 to U2, U23 to U20, U24 to U21, U25 to U22, U26 to U23, U51 to U24, U54 to U26, U28 to U27, U29 to U28, U30 to U29, U5 to U3, U31 to U30, U32 to U31, U33 to U32, U36 to U34, U37 to U35, U38 to U36, U39 to U37, U40 to U38, U41 to U39, U6 to U4, U19 to U40, U27 to U41, U44 to U42, U45 to U43, U46 to U44, U47 to U45, U48 to U46, U34 to U47, U35 to U48, U1 to U49, U7 to U5, U49 to U51, U42 to U52, U43 to U53, U52 to U54, U53 to U55, U8 to U6, U2 to U7, U9 to U8, U10 to U9
Connections:
- net +3V3: now also C37.1, R70.1, R87.1, R94.1, U25.14 (VCC), U33.8 (VCC)
- net +5V_USB: now also C36.1, D33.1 (A1), F3.1; no longer J2.A4 (VBUS), J2.A9 (VBUS), J2.B4 (VBUS), J2.B9 (VBUS)
- net A+_OUT: now also A1.1, D34.2 (A2), R95.1, U33.6 (A)
- net B-_OUT: now also D34.1 (A1), R94.2, R96.2, U33.7 (B)
- net GND: now also C35.2, C36.2, C37.2, D33.2 (A2), D34.3 (common), R95.2, U25.7 (GND), U33.5 (GND)
- net RS485_RXD0: now also U25.4
- net RS485_TXD0: now also R70.2, U25.1
- net at U40.5 (UD+): now also J2.A6 (D+), J2.B6 (D+)
- net at U40.6 (UD-): now also J2.A7 (D-), J2.B7 (D-)
- new net: D32.1 (K), R84.2, U25.10, U33.4 (DI)
- new net: U25.11, U25.2
- new net: C35.1, D32.2 (A), R84.1, U25.13
- new net: U25.3, U25.8
- new net: R87.2, U25.9, U33.1 (RO)
- new net: U25.12, U33.2 (~{RE}), U33.3 (DE)
- new net: F3.2, J2.A4 (VBUS), J2.A9 (VBUS), J2.B4 (VBUS), J2.B9 (VBUS)
- new net: A1.2, R96.1
Other:
- note added: "MCP23017"
- note added: "MCP_A"
- note added: "MCP_B"
- note removed: "ADC"
- note removed: "Input Board v0.4 ESP"
- note removed: "MCP23017 and PCF8575"
- note removed: "PINOUT"
- note removed: "WT32- ETH01"
- title: Input Board ESP -> (none)
- moved on the sheet: A2, A3, A4, A5, A6, A7, A8, BT1, C1, C10, C11, C12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
