File: boneIO - input WT32.kicad_sch (KiCad schematic)
At the start: 340 parts, among them J1 P1, J10 RX, J11 USB_C_Receptacle_USB2.0, J12 UART, J13 Conn_02x04_Odd_Even, J14 EXT_PSU, J2 P2, J3 POWER, J4 P4, J5 P3, J6 P5, J7 P6, J8 P7, J9 TX, Q1 AO3401A, Q3 BC817, Q4 BC817, SW1 USER_SWITCH, SW2 SW_DIP_x04, U1 EL357N, U10 WT32-ETH01, U11 INA219AxD, U12 EL357N, U13 EL357N, U14 EL357N, U15 EL357N, U16 EL357N, U17 EL357N, U18 XL1509-5, U19 EL357N, U2 EL357N, U20 EL357N, U21 EL357N, U22 EL357N, U23 EL357N, U24 EL357N, U25 RT9013-33GB, U26 EL357N, U27 EL357N, U28 EL357N, U29 SN74LVC1G3157, U3 EL357N, U30 EL357N, U31 EL357N, U32 EL357N, U33 EL357N, U34 EL357N, U35 EL357N, U36 SN74LVC1G3157, U37 RS485, U38 CH340C, U39 EL357N, U4 EL357N, U40 EL357N, U41 EL357N, U42 EL357N, U43 EL357N, U44 2N7002DW/BSS138PS, U45 2N7002DW/BSS138PS, U46 MCP23017_SS, U47 DS1307Z+, U48 SN65HVD230, U49 MCP23017_SS, U5 EL357N, U50 PCA9515, U51 PCA9515, U6 EL357N, U7 EL357N, U8 EL357N, U9 EL357N, Y1 32,788 MHz

Commit message: input board ESP v0.4
added USB protection
Parts:
- added C34: 100n, Capacitor_SMD:C_0603_1608Metric, symbol Device:C
- added D33: 5V6, Diode_SMD:D_MiniMELF, symbol Device:D_Zener_ALT
- added F3: 6V 500mA, Fuse:Fuse_1206_3216Metric, symbol Device:Fuse
- renumbered C4 to C1, C13 to C10, C14 to C11, C15 to C12, C16 to C13, C17 to C14, C18 to C15, C19 to C16, C20 to C17, C21 to C18, C22 to C19, C5 to C2, C23 to C20, C24 to C21, C25 to C22, C26 to C23, C27 to C24, C28 to C25, C29 to C26, C30 to C27, C31 to C28, C32 to C29, C6 to C3, C33 to C30, C3 to C31, C2 to C32, C1 to C33, C40 to C35, C34 to C36, C35 to C37, C36 to C38, C37 to C39, C7 to C4, C38 to C40, C39 to C41, C41 to C42, C42 to C43, C43 to C44, C44 to C45, C45 to C46, C46 to C47, C8 to C5, C47 to C51, C51 to C54, C9 to C6, C10 to C7, C11 to C8, C12 to C9, D4 to D1, D13 to D10, D14 to D11, D15 to D12, D16 to D13, D17 to D14, D18 to D15, D19 to D16, D20 to D17, D21 to D18, D22 to D19, D5 to D2, D23 to D20, D24 to D21, D25 to D22, D26 to D23, D27 to D24, D28 to D25, D29 to D26, D30 to D27, D31 to D28, D32 to D29, D6 to D3, D3 to D30, D2 to D31, D1 to D32, D33 to D34, D34 to D35, D35 to D36, D36 to D37, D37 to D38, D38 to D39, D7 to D4, D39 to D40, D40 to D41, D41 to D42, D42 to D43, D43 to D44, D44 to D45, D45 to D46, D46 to D47, D47 to D48, D48 to D49, D8 to D5, D9 to D6, D10 to D7, D11 to D8, D12 to D9, Q3 to Q2, Q4 to Q3, R10 to R1, R19 to R10, R99 to R100, R100 to R101, R108 to R102, R109 to R103, R103 to R104, R104 to R105, R105 to R106, R106 to R107, R107 to R108, R110 to R109, R20 to R11, R111 to R110, R112 to R111, R113 to R112, R114 to R113, R115 to R114, R116 to R115, R117 to R116, R118 to R117, R119 to R118, R122 to R119, R21 to R12, R125 to R120, R126 to R121, R132 to R122, R133 to R123, R134 to R124, R127 to R125, R128 to R126, R129 to R127, R130 to R128, R131 to R129, R22 to R13, R135 to R130, R137 to R131, R120 to R132, R121 to R133, R123 to R134, R124 to R135, R142 to R136, R143 to R137, R141 to R138, R144 to R139, R23 to R14, R145 to R140, R136 to R141, R138 to R142, R139 to R143, R140 to R144, R146 to R145, R147 to R146, R24 to R15, R25 to R16, R26 to R17, R27 to R18, R28 to R19, R11 to R2, R29 to R20, R30 to R21, R31 to R22, R32 to R23, R33 to R24, R34 to R25, R35 to R26, R36 to R27, R37 to R28, R38 to R29, R12 to R3, R39 to R30, R40 to R31, R41 to R32, R42 to R33, R43 to R34, R44 to R35, R45 to R36, R46 to R37, R47 to R38, R48 to R39, R13 to R4, R49 to R40, R50 to R41, R51 to R42, R52 to R43, R53 to R44, R54 to R45, R55 to R46, R56 to R47, R57 to R48, R58 to R49, R14 to R5, R59 to R50, R60 to R51, R61 to R52, R62 to R53, R63 to R54, R64 to R55, R65 to R56, R66 to R57, R67 to R58, R68 to R59, R15 to R6, R69 to R60, R80 to R61, R70 to R62, R71 to R63, R72 to R64, R73 to R65, R7 to R66, R4 to R67, R1 to R68, R88 to R69, R16 to R7, R74 to R70, R75 to R71, R76 to R72, R8 to R73, R5 to R74, R2 to R75, R77 to R76, R78 to R77, R79 to R78, R9 to R79, R17 to R8, R6 to R80, R3 to R81, R101 to R82, R102 to R83, R82 to R84, R83 to R85, R84 to R86, R85 to R87, R86 to R88, R87 to R89, R18 to R9, R89 to R90, R90 to R91, R91 to R92, R92 to R93, R93 to R94, R94 to R95, R95 to R96, R96 to R97, R97 to R98, R98 to R99, U4 to U1, U13 to U10, U14 to U11, U15 to U12, U16 to U13, U17 to U14, U18 to U15, U19 to U16, U20 to U17, U21 to U18, U22 to U19, U5 to U2, U23 to U20, U24 to U21, U25 to U22, U29 to U23, U26 to U24, U27 to U25, U28 to U26, U3 to U27, U2 to U28, U1 to U29, U6 to U3, U36 to U30, U38 to U31, U30 to U32, U31 to U33, U32 to U34, U33 to U35, U34 to U36, U35 to U37, U37 to U38, U7 to U4, U47 to U46, U48 to U47, U46 to U48, U50 to U49, U8 to U5, U51 to U50, U49 to U51, U9 to U6, U10 to U7, U11 to U8, U12 to U9
Connections:
- net +5V_USB: now also C34.1, D33.1 (K), F3.2; no longer J11.A4 (VBUS), J11.A9 (VBUS), J11.B4 (VBUS), J11.B9 (VBUS)
- net GND: now also C34.2, D33.2 (A)
- new net: F3.1, J11.A4 (VBUS), J11.A9 (VBUS), J11.B4 (VBUS), J11.B9 (VBUS)
Other:
- moved on the sheet: J11, J12, L3

Commit message: v0.4
najnowsza wersja input board ESP
Parts:
- removed A0_2, A1_1, A1_2, A2_1, A2_2, CAN_T1: Opened, Jumper:SolderJumper-2_P1.3mm_Open_RoundedPad1.0x1.5mm, symbol ESP32-EVB_Rev_I:SJ
- removed C25, C27: 1uF, Capacitor_SMD:C_0805_2012Metric, symbol Device:C
- removed C34, C48: 100n, Capacitor_SMD:C_0603_1608Metric, symbol Device:C
- removed D10, D33: 5V6, Diode_SMD:D_MiniMELF, symbol Device:D_Zener_ALT
- removed D8: BAT54A, Package_TO_SOT_SMD:SOT-23, symbol Diode:BAT54A
- removed D9: LED_GREEN, LED_SMD:LED_0805_2012Metric, symbol Device:LED_ALT
- removed F3: 6V 500mA, Fuse:Fuse_1206_3216Metric, symbol Device:Fuse
- removed FID1, FID2: Fiducial, Fiducial:Fiducial_0.5mm_Mask1.5mm, symbol Mechanical:Fiducial
- removed J10: RX, Connector_PinHeader_2.54mm:PinHeader_1x03_P2.54mm_Vertical, symbol Connector:Screw_Terminal_01x03
- removed J9: TX, Connector_PinHeader_2.54mm:PinHeader_1x03_P2.54mm_Vertical, symbol Connector:Screw_Terminal_01x03
- removed R123: 4.7k, Resistor_SMD:R_0603_1608Metric, symbol Device:R
- removed R125: 10k, Resistor_SMD:R_0603_1608Metric, symbol Device:R
- removed U45: 2N7002DW/BSS138PS, Package_TO_SOT_SMD:SOT-363_SC-70-6, symbol Transistor_FET:2N7002DW
- added A1, A2, A3, A5, A6, A7: Opened, Jumper:SolderJumper-2_P1.3mm_Open_RoundedPad1.0x1.5mm, symbol ESP32-EVB_Rev_I:SJ
- added C10: 4.7n, Capacitor_SMD:C_0603_1608Metric, symbol Device:C
- added C29, C31: 10u, Capacitor_SMD:C_1206_3216Metric, symbol Device:C
- added C38: 100n, Capacitor_SMD:C_0603_1608Metric, symbol Device:C
- added D1: SMBJ28CA, Diode_SMD:D_SMB, symbol Diode:SM6T18A
- added D10: SMBJ5.0A, Diode_SMD:D_SMB, symbol Diode:SM6T18A
- added D27, D28: LED_GREEN, LED_SMD:LED_0805_2012Metric, symbol Device:LED_ALT
- added L10, L11: BLM21_NC, Inductor_SMD:L_0805_2012Metric, symbol Device:L_Small
- added L8, L9: BLM21PG121SN1D, Inductor_SMD:L_0805_2012Metric, symbol Device:L_Small
- added R32: 1M, Resistor_SMD:R_0603_1608Metric, symbol Device:R
- added R54: 0k, Resistor_SMD:R_0603_1608Metric, symbol Device:R
- added R73, R74: 1.2k, Resistor_SMD:R_0603_1608Metric, symbol Device:R
- added U18: USBLC6-2SC6, Package_TO_SOT_SMD:SOT-23-6, symbol Power_Protection:USBLC6-2SC6
- added U27: LM358, Package_SO:SOIC-8_3.9x4.9mm_P1.27mm, symbol Amplifier_Operational:LM358_K
- added U50, U52: PCF8575, Package_SO:SSOP-24_5.3x8.2mm_P0.65mm, symbol Interface_Expansion:PCF8575
- C9: value 100n -> 10u; footprint Capacitor_SMD:C_0603_1608Metric -> Capacitor_SMD:C_1206_3216Metric; JLCPCB (none) -> C107149
- D19: value B5819WS -> B5819W
- D31: renamed from D29; value LED -> LED N
- F1: footprint Fuse:Fuse_2512_6332Metric -> Fuse:Fuse_1812_4532Metric
- J2: renamed from J11; value USB_C_Receptacle_USB2.0 -> GT-USB-7010AN
- L1: footprint Inductor_SMD:L_10.4x10.4_H4.8 -> Inductor_SMD:L_7.3x7.3_H4.5
- Q2, Q3: value BC817 -> SS8050
- R114: renamed from R96; value 680R -> 1.2k
- R115: renamed from R97; value 680R -> 1.2k
- R116: renamed from R98; value 680R -> 1.2k
- R117: renamed from R99; value 680R -> 1.2k
- R118: renamed from R100; value 680R -> 1.2k
- R119: renamed from R101; value 680R -> 1.2k
- R133: renamed from R114; value 680R -> 1.2k
- R135: renamed from R115; value 680R -> 1.2k
- R136: renamed from R116; value 680R -> 1.2k
- R137: renamed from R117; value 680R -> 1.2k
- R138: renamed from R118; value 680R -> 1.2k
- R17: renamed from R13; value 680R -> 1.2k
- R18: renamed from R14; value 680R -> 1.2k
- R19: renamed from R15; value 680R -> 1.2k
- R20: renamed from R16; value 680R -> 1.2k
- R21: renamed from R17; value 680R -> 1.2k
- R22: renamed from R18; value 680R -> 1.2k
- R25: renamed from R19; value 100R_1% -> 0.1R_1%
- R41: renamed from R35; value 680R -> 1.2k
- R42: renamed from R36; value 680R -> 1.2k
- R43: renamed from R37; value 680R -> 1.2k
- R44: renamed from R38; value 680R -> 1.2k
- R45: renamed from R39; value 680R -> 1.2k
- R46: renamed from R40; value 680R -> 1.2k
- R55: renamed from R41; value 330R -> 1.2k
- R62: renamed from R55; value 680R -> 1.2k
- R63: renamed from R56; value 680R -> 1.2k
- R64: renamed from R57; value 680R -> 1.2k
- R65: renamed from R58; value 680R -> 1.2k
- R66: renamed from R59; value 680R -> 1.2k
- R67: renamed from R60; value 680R -> 1.2k
- R68: renamed from R127; value 1,5k -> 1.2k
- R71: renamed from R129; value 10k -> 15k
- R81: renamed from R62; value 330R -> 1.2k
- R86: renamed from R72; value 10k -> 10kN
- R90: renamed from R76; value 680R -> 1.2k
- R91: renamed from R77; value 680R -> 1.2k
- R92: renamed from R78; value 680R -> 1.2kN
- R93: renamed from R79; value 680R -> 1.2k
- R94: renamed from R80; value 680R -> 1.2k
- R95: renamed from R81; value 680R -> 1.2k
- RV1: footprint Varistor:RV_Disc_D7mm_W3.5mm_P5mm -> Resistor_THT:R_Axial_DIN0204_L3.6mm_D1.6mm_P5.08mm_Vertical
- renumbered A0_1 to A4, C50 to C1, C17 to C11, C10 to C12, C11 to C13, C12 to C14, C13 to C15, C14 to C16, C15 to C17, C8 to C18, C16 to C19, C1 to C2, C35 to C20, C18 to C21, C19 to C22, C20 to C23, C21 to C24, C22 to C25, C23 to C26, C24 to C27, C42 to C28, C2 to C3, C26 to C30, C28 to C32, C29 to C33, C30 to C34, C31 to C35, C32 to C36, C33 to C37, C49 to C39, C3 to C4, C36 to C40, C37 to C41, C38 to C42, C39 to C43, C40 to C44, C41 to C45, C53 to C46, C52 to C47, C43 to C48, C44 to C49, C4 to C5, C45 to C50, C46 to C51, C47 to C52, C51 to C53, C5 to C6, C6 to C7, C7 to C8, D12 to D11, D13 to D12, D14 to D13, D15 to D14, D16 to D15, D17 to D16, D11 to D17, D1 to D2, D27 to D29, D46 to D3, D28 to D30, D30 to D32, D31 to D33, D32 to D34, D47 to D35, D48 to D36, D34 to D37, D35 to D38, D36 to D39, D2 to D4, D37 to D40, D38 to D41, D39 to D42, D45 to D43, D49 to D44, D40 to D45, D41 to D46, D42 to D47, D43 to D48, D44 to D49, D3 to D5, D4 to D6, D5 to D7, D6 to D8, D7 to D9, J3 to J1, J6 to J10, J7 to J11, J8 to J12, J12 to J3, J14 to J4, J13 to J5, J1 to J6, J2 to J7, J4 to J8, J5 to J9, R131 to R1, R7 to R10, R84 to R100, R85 to R101, R86 to R102, R87 to R103, R88 to R104, R89 to R105, R124 to R106, R130 to R107, R90 to R108, R91 to R109, R8 to R11, R92 to R110, R93 to R111, R94 to R112, R95 to R113, R9 to R12, R138 to R120, R140 to R121, R104 to R122, R105 to R123, R106 to R124, R107 to R125, R108 to R126, R145 to R127, R109 to R128, R110 to R129, R10 to R13, R111 to R130, R112 to R131, R113 to R132, R146 to R134, R132 to R139, R11 to R14, R133 to R140, R134 to R141, R135 to R142, R141 to R143, R61 to R144, R143 to R145, R144 to R146, R142 to R147, R69 to R148, R12 to R15, R139 to R16, R1 to R2, R20 to R23, R21 to R24, R22 to R26, R23 to R27, R24 to R28, R25 to R29, R2 to R3, R26 to R30, R27 to R31, R82 to R33, R29 to R34, R30 to R35, R31 to R36, R32 to R37, R33 to R38, R34 to R39, R3 to R4, R83 to R40, R28 to R47, R42 to R48, R43 to R49, R4 to R5, R44 to R50, R45 to R51, R46 to R52, R47 to R53, R49 to R56, R50 to R57, R51 to R58, R52 to R59, R5 to R6, R53 to R60, R54 to R61, R102 to R69, R6 to R7, R103 to R70, R48 to R72, R63 to R75, R64 to R76, R65 to R77, R66 to R78, R67 to R79, R136 to R8, R68 to R80, R128 to R82, R126 to R83, R70 to R84, R71 to R85, R73 to R87, R74 to R88, R75 to R89, R137 to R9, R119 to R96, R121 to R97, R120 to R98, R122 to R99, SW2 to SW1, SW1 to SW2, U47 to U1, U9 to U10, U10 to U11, U11 to U12, U12 to U13, U13 to U14, U14 to U15, U38 to U16, U15 to U17, U31 to U19, U7 to U2, U16 to U20, U17 to U21, U18 to U22, U19 to U23, U20 to U24, U21 to U25, U22 to U26, U24 to U28, U25 to U29, U1 to U3, U26 to U30, U27 to U31, U28 to U32, U29 to U33, U44 to U34, U46 to U35, U32 to U36, U33 to U37, U34 to U38, U35 to U39, U2 to U4, U36 to U40, U37 to U41, U49 to U42, U50 to U43, U39 to U44, U40 to U45, U41 to U46, U42 to U47, U43 to U48, U48 to U49, U3 to U5, U23 to U51, U51 to U53, U30 to U54, U4 to U6, U5 to U7, U6 to U8, U8 to U9
Connections:
- net 1-WIRE_OUT is gone; now on net 1-WIRE: J11.7 (Pin_7), R98.2
- net +3V3: now also J11.4 (Pin_4), C31.1, D27.2 (A), D28.2 (A); no longer A4.2, C53.1, C54.1, C8.2, J11.5 (Pin_5), R10.2, R108.2, R109.2, R11.2, R110.2, R111.2, R112.2, R113.2, R114.2, R115.2, R116.2, R117.2, R118.2, R119.2, R12.2, R128.2, R129.2, R13.2, R130.2, R131.2, R132.2, R133.2, R135.2, R136.2, R137.2, R138.2, R14.2, R142.1, R147.1, R15.2, R17.2, R18.2, R19.2, R20.2, R21.2, R22.2, R34.2, R35.2, R36.2, R37.2, R38.2, R39.2, R41.2, R42.2, R43.2, R44.2, R45.2, R46.2, R56.2, R57.2, R58.2, R59.2, R60.2, R61.2, R62.2, R63.2, R64.2, R65.2, R66.2, R67.2, R84.2, R85.2, R86.2, R87.2, R88.2, R89.2, R90.2, R91.2, R92.2, R93.2, R94.2, R95.2, U49.9 (VDD), U53.9 (VDD), U9.5 (VS)
- net +5V: now also A4.2, C53.1, C54.1, C8.2, R10.2, R108.2, R109.2, R11.2, R110.2, R111.2, R112.2, R113.2, R114.2, R115.2, R116.2, R117.2, R118.2, R119.2, R12.2, R128.2, R129.2, R13.2, R130.2, R131.2, R132.2, R133.2, R135.2, R136.2, R137.2, R138.2, R14.2, R142.1, R147.1, R15.2, R17.2, R18.2, R19.2, R20.2, R21.2, R22.2, R34.2, R35.2, R36.2, R37.2, R38.2, R39.2, R41.2, R42.2, R43.2, R44.2, R45.2, R46.2, R56.2, R57.2, R58.2, R59.2, R60.2, R61.2, R62.2, R63.2, R64.2, R65.2, R66.2, R67.2, R84.2, R85.2, R86.2, R87.2, R88.2, R89.2, R90.2, R91.2, R92.2, R93.2, R94.2, R95.2, U49.9 (VDD), U53.9 (VDD), U9.5 (VS), A2.2, A3.2, A5.2, A6.2, A7.2, C29.1, C38.1, U27.8 (VCC), U50.24 (VDD), U52.24 (VDD)
- net +5V_USB: now also J2.A4 (VBUS), J2.A9 (VBUS), J2.B4 (VBUS), J2.B9 (VBUS), U18.2 (GND)
- net CAN_H: now also R16.2
- net CAN_L: now also A1.1; no longer R16.1
- net CH_RXD: now also U19.2 (TXD); no longer U19.3 (RXD)
- net CH_TXD: now also U19.3 (RXD); no longer U19.2 (TXD)
- net EX_IO12: now also D31.1 (K), R86.1, U30.4; no longer R68.1, R71.1
- net EX_IO17: now also D30.1 (K), R85.1, U29.4; no longer J11.6 (Pin_6)
- net EX_IO2: now also J11.5 (Pin_5); no longer R82.1, R83.1
- net EX_IO36: now also R68.1, R71.1; no longer D30.1 (K), R85.1, U29.4
- net EX_IO39: now also R82.1, R83.1; no longer D31.1 (K), R86.1, U30.4
- net GND: now also J11.6 (Pin_6), J2.A1 (GND), J2.A12 (GND), J2.B1 (GND), J2.B12 (GND), SW1.4, C10.2, C29.2, C31.2, C38.2, D10.2 (A2), R32.2, R54.1, U18.5 (VBUS), U27.4 (GND), U50.12 (VSS), U52.12 (VSS); no longer J11.2 (Pin_2), J5.1 (Pin_1), J5.3 (Pin_3), L3.1, SW1.8
- net GND1: now also SW1.3; no longer SW1.7
- net GNDA: now also L10.1, L9.2; no longer L5.1, L6.1, SW1.1, SW1.2
- net GNDS: now also L3.1, D1.2 (A2)
- net GND_RS485: now also R54.2
- net I2C_SCL: no longer U49.12 (SCK), U53.12 (SCK), U9.4 (SCL)
- net I2C_SCL_HV: now also U49.12 (SCK), U53.12 (SCK), U9.4 (SCL), U50.22 (SCL), U52.22 (SCL)
- net I2C_SDA: no longer U49.13 (SDA), U53.13 (SDA), U9.3 (SDA)
- net I2C_SDA_HV: now also U49.13 (SDA), U53.13 (SDA), U9.3 (SDA), U50.23 (SDA), U52.23 (SDA)
- net IO1_TXD0: now also R73.1
- net IO3_RXD0: now also R74.1
- net MCP_1: now also U50.4 (P00)
- net MCP_10: now also U50.14 (P11)
- net MCP_11: now also U50.15 (P12)
- net MCP_12: now also U50.16 (P13)
- net MCP_13: now also U50.17 (P14)
- net MCP_14: now also U50.18 (P15)
- net MCP_15: now also U50.19 (P16)
- net MCP_16: now also U50.20 (P17)
- net MCP_17: now also U52.11 (P07)
- net MCP_18: now also U52.10 (P06)
- net MCP_19: now also U52.9 (P05)
- net MCP_2: now also U50.5 (P01)
- net MCP_20: now also U52.8 (P04)
- net MCP_21: now also U52.7 (P03)
- net MCP_22: now also U52.6 (P02)
- net MCP_23: now also U52.5 (P01)
- net MCP_24: now also U52.4 (P00)
- net MCP_25: now also U52.13 (P10)
- net MCP_26: now also U52.14 (P11)
- net MCP_27: now also U52.15 (P12)
- net MCP_28: now also U52.16 (P13)
- net MCP_29: now also U52.17 (P14)
- net MCP_3: now also U50.6 (P02)
- net MCP_30: now also U52.18 (P15)
- net MCP_31: now also U52.19 (P16)
- net MCP_32: now also U52.20 (P17)
- net MCP_4: now also U50.7 (P03)
- net MCP_5: now also U50.8 (P04)
- net MCP_6: now also U50.9 (P05)
- net MCP_7: now also U50.10 (P06)
- net MCP_8: now also U50.11 (P07)
- net MCP_9: now also U50.13 (P10)
- net VCC: no longer RV1.1
- net VDD: now also L10.2, L8.2; no longer L4.2, L7.2, SW1.3, SW1.4
- net IN_2: now reaches R147.2, U53.18 (~{RESET})
- net IN_2: now also U52.1 (INT)
- net at C11.1, F2.1, U2.25 (5V): now also D10.1 (A1)
- net A0_1: now reaches A4.1, R141.1, U49.15 (A0)
- net A0_1: now also U50.21 (A0)
- net A1_1: now reaches R140.1, U49.16 (A1)
- net A1_1: now also A3.1, U50.2 (A1)
- net A2_1: now reaches R139.1, U49.17 (A2)
- net A2_1: now also A2.1, U50.3 (A2)
- net IN_1: now reaches R142.2, U49.18 (~{RESET})
- net IN_1: now also U50.1 (INT)
- net A0_2: now reaches R146.1, U53.15 (A0)
- net A0_2: now also A7.1, U52.21 (A0)
- net at D35.1 (K), L4.1: now also SW1.2; no longer SW1.6
- net A2_2: now reaches R143.1, U53.17 (A2)
- net A2_2: now also A5.1, U52.3 (A2)
- net at D36.1 (K), L7.1: now also SW1.1; no longer SW1.5
- net at J2.A6 (D+), J2.B6 (D+): now also U18.3 (I/O2); no longer U19.5 (UD+)
- net at J2.A7 (D-), J2.B7 (D-): now also U18.1 (I/O1); no longer U19.6 (UD-)
- net A1_2: now reaches R145.1, U53.16 (A1)
- net A1_2: now also A6.1, U52.2 (A1)
- net at D2.2 (A), F1.1: now also RV1.1, D1.1 (A1)
- net ADC_1: no longer names the net of R82.2
- net ADC_1: now also U27.6 (2IN-), U27.7 (2OUT); no longer J11.4 (Pin_4)
- net ADC_2: no longer names the net of R71.2
- net ADC_2: now also U27.1 (1OUT), U27.2 (1IN-); no longer J11.3 (Pin_3)
- net GPIO36_OUT renamed GPIO17_OUT
- net GPIO39_OUT renamed GPIO12_OUT
- new net: D28.1 (K), R74.2
- new net: A1.2, R16.1
- new net: C10.1, J2.S1 (SHIELD), R32.1
- new net: U18.4 (I/O2), U19.5 (UD+)
- new net: U18.6 (I/O1), U19.6 (UD-)
- new net: D27.1 (K), R73.2
- new net A0: J11.2 (Pin_2), U27.3 (1IN+)
- new net A1: J11.3 (Pin_3), U27.5 (2IN+)
- new net Earth: J5.1 (Pin_1), J5.3 (Pin_3), L3.2
- new net GND2: L11.2, L5.1, L6.1, L9.1, SW1.5, SW1.6
- new net VDD_AA: L11.1, L4.2, L7.2, L8.1, SW1.7, SW1.8
- no-connect marks 11 -> 13
Other:
- note added: "ADC"
- note added: "After connecting the USB, the pins are set to programming, after disconnecting the USB, the pins are set to RS485"
- note added: "Automatic UART switching"
- note added: "INA219"
- note added: "Input Board v0.4 ESP"
- note added: "Logic Converter"
- note added: "MCP23017 and PCF8575"
- note added: "PINOUT"
- note added: "WT32- ETH01"
- note added: "address: 0x26"
- note added: "address: 0x27"
- note added: "address: 0x40"
- note added: "address: 0x68"
- note added: "module TTL RS485"
- note removed: "MCP23017"
- note removed: "RS485"
- title: (none) -> Input Board ESP
- moved on the sheet: A4, BT1, C1, C11, C12, C13, C14, C15, C16, C17, C18, C19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

Commit message: input_board_v0.5
1. Remove internal dip switch and EXT PSU connector
2. adding an external dip switch in place of the EXT PSU connector for switching input control ( +24v or GND)
3. adding 2 i2c buses. 1 bus is responsible for input and 2 for output
4. addition of PCF8574 for inputs and MENU button
5. corrected ADC.
Parts:
- removed A1, A2, A3, A4, A5, A6, A7: Opened, Jumper:SolderJumper-2_P1.3mm_Open_RoundedPad1.0x1.5mm, symbol ESP32-EVB_Rev_I:SJ
- removed C38: 100n, Capacitor_SMD:C_0603_1608Metric, symbol Device:C
- removed D35, D36: B5819W, Diode_SMD:D_SOD-123, symbol Device:D_ALT
- removed J4: EXT_PSU, Connector_Phoenix_MSTB:PhoenixContact_MSTBA_2,5_2-G_1x02_P5.00mm_Horizontal, symbol Connector:Screw_Terminal_01x02
- removed L10, L11, L4, L5, L6, L7: BLM21_NC, Inductor_SMD:L_0805_2012Metric, symbol Device:L_Small
- removed L8, L9: BLM21PG121SN1D, Inductor_SMD:L_0805_2012Metric, symbol Device:L_Small
- removed R139, R140, R141, R143, R145: 10k, Resistor_SMD:R_0603_1608Metric, symbol Device:R
- removed R47, R72, R82: 100k, Resistor_SMD:R_0603_1608Metric, symbol Device:R
- removed R54: 0k, Resistor_SMD:R_0603_1608Metric, symbol Device:R
- removed R68: 1.2k, Resistor_SMD:R_0603_1608Metric, symbol Device:R
- removed R71, R83: 15k, Resistor_SMD:R_0603_1608Metric, symbol Device:R
- removed SW1: SW_DIP_x04, Button_Switch_SMD:SW_DIP_SPSTx04_Slide_Omron_A6S-410x_W8.9mm_P2.54mm, symbol Switch:SW_DIP_x04
- removed U18: USBLC6-2SC6, Package_TO_SOT_SMD:SOT-23-6, symbol Power_Protection:USBLC6-2SC6
- removed U27: LM358, Package_SO:SOIC-8_3.9x4.9mm_P1.27mm, symbol Amplifier_Operational:LM358_K
- removed U43: PCA9515, Package_SO:SO-8_3.9x4.9mm_P1.27mm, symbol Interface_Expansion:PCA9515
- added BZ1: Buzzer, Library2:XDCR_KXG0909P, symbol Device:Buzzer
- added C35, C57: 100n, Capacitor_SMD:C_0603_1608Metric, symbol Device:C
- added C43, C45: 10p, Capacitor_SMD:C_0603_1608Metric, symbol Device:C
- added D33: SMBJ5.0A, Diode_SMD:D_SMB, symbol Diode:SM6T18A
- added D34, D41: BAT54S, Package_TO_SOT_SMD:SOT-23, symbol Diode:BAT54S
- added D9: 1N4148, Diode_SMD:D_MiniMELF, symbol Device:D
- added F3: 6V 500mA, Fuse:Fuse_1206_3216Metric, symbol Device:Fuse
- added Q1: BC817, Package_TO_SOT_SMD:SOT-23, symbol Transistor_BJT:BC817
- added R1, R22, R8: 10k, Resistor_SMD:R_0603_1608Metric, symbol Device:R
- added R111, R95: 30k, Resistor_SMD:R_0603_1608Metric, symbol Device:R
- added R112, R136, R32, R39, R96: 4.7k, Resistor_SMD:R_0603_1608Metric, symbol Device:R
- added R132, R133: 100R, Resistor_SMD:R_0603_1608Metric, symbol Device:R
- added R148, R149: 330R, Resistor_SMD:R_1206_3216Metric, symbol Device:R
- added R15: 1.2k, Resistor_SMD:R_0603_1608Metric, symbol Device:R
- added SW2: SW_DIP_x04, Button_Switch_THT:SW_DIP_SPSTx04_Piano_10.8x11.72mm_W7.62mm_P2.54mm, symbol Switch:SW_DIP_x04
- added U52: PCF8574TS, Package_SO:SSOP-20_5.3x7.2mm_P0.65mm, symbol Interface_Expansion:PCF8574TS
- C26: renamed from C30; value 460p -> 470p
- C9: value 10u -> 10uF; footprint Capacitor_SMD:C_1206_3216Metric -> Capacitor_SMD:C_0603_1608Metric
- D29: renamed from D31; value LED N -> LED
- D42: renamed from D27; footprint LED_SMD:LED_0805_2012Metric -> LED_SMD:LED_0603_1608Metric
- D43: renamed from D28; footprint LED_SMD:LED_0805_2012Metric -> LED_SMD:LED_0603_1608Metric
- F1: value Fuse 2A -> MF-MSMF075/24-2
- Q3: renamed from Q2; value SS8050 -> BC817
- Q4: renamed from Q3; value SS8050 -> BC817
- R146: value 10k -> 4.7k
- R77: renamed from R86; value 10kN -> 10k
- R83: renamed from R92; value 1.2kN -> 1.2k
- renumbered C2 to C1, C12 to C10, C13 to C11, C14 to C12, C15 to C13, C16 to C14, C17 to C15, C11 to C16, C19 to C17, C21 to C18, C22 to C19, C3 to C2, C23 to C20, C24 to C21, C25 to C22, C26 to C23, C27 to C24, C29 to C25, C31 to C27, C32 to C28, C33 to C29, C4 to C3, C34 to C30, C35 to C31, C36 to C32, C37 to C33, C10 to C34, C40 to C36, C41 to C37, C42 to C38, C43 to C39, C5 to C4, C44 to C40, C45 to C41, C20 to C42, C28 to C44, C48 to C46, C49 to C47, C50 to C48, C51 to C49, C6 to C5, C52 to C50, C39 to C51, C1 to C52, C47 to C54, C46 to C55, C54 to C56, C7 to C6, C8 to C7, C18 to C8, D17 to D11, D11 to D12, D12 to D13, D13 to D14, D14 to D15, D15 to D16, D16 to D17, D29 to D27, D30 to D28, D4 to D3, D32 to D30, D33 to D31, D34 to D32, D37 to D35, D38 to D36, D39 to D37, D40 to D38, D41 to D39, D5 to D4, D42 to D40, D45 to D44, D46 to D45, D47 to D46, D48 to D47, D49 to D48, D43 to D49, D6 to D5, D3 to D50, D44 to D51, D7 to D6, D8 to D7, D9 to D8, J11 to J10, J12 to J11, J6 to J4, J7 to J5, J5 to J6, J8 to J7, J9 to J8, J10 to J9, Q1 to Q2, R11 to R10, R111 to R100, R112 to R101, R113 to R102, R114 to R103, R115 to R104, R116 to R105, R117 to R106, R118 to R107, R119 to R108, R69 to R109, R12 to R11, R70 to R110, R122 to R113, R123 to R114, R124 to R115, R125 to R116, R126 to R117, R73 to R118, R74 to R119, R13 to R12, R128 to R120, R129 to R121, R130 to R122, R131 to R123, R132 to R124, R133 to R125, R135 to R126, R136 to R127, R137 to R128, R138 to R129, R14 to R13, R96 to R130, R97 to R131, R99 to R134, R98 to R135, R106 to R137, R107 to R138, R1 to R139, R15 to R14, R142 to R140, R8 to R141, R9 to R142, R16 to R143, R120 to R144, R121 to R145, R127 to R150, R134 to R151, R17 to R16, R18 to R17, R19 to R18, R20 to R19, R21 to R20, R22 to R21, R25 to R23, R23 to R24, R24 to R25, R34 to R33, R35 to R34, R36 to R35, R37 to R36, R38 to R37, R39 to R38, R41 to R40, R42 to R41, R43 to R42, R44 to R43, R45 to R44, R46 to R45, R55 to R46, R48 to R47, R49 to R48, R50 to R49, R51 to R50, R52 to R51, R53 to R52, R144 to R53, R56 to R54, R57 to R55, R58 to R56, R59 to R57, R60 to R58, R61 to R59, R62 to R60, R63 to R61, R64 to R62, R65 to R63, R66 to R64, R67 to R65, R81 to R66, R148 to R67, R75 to R68, R76 to R69, R77 to R70, R78 to R71, R79 to R72, R80 to R73, R32 to R74, R84 to R75, R85 to R76, R87 to R78, R88 to R79, R89 to R80, R90 to R81, R91 to R82, R93 to R84, R94 to R85, R95 to R86, R33 to R87, R40 to R88, R100 to R89, R10 to R9, R101 to R90, R102 to R91, R103 to R92, R104 to R93, R105 to R94, R108 to R97, R109 to R98, R110 to R99, SW2 to SW1, U3 to U1, U11 to U10, U12 to U11, U13 to U12, U14 to U13, U15 to U14, U17 to U15, U20 to U17, U21 to U18, U22 to U19, U4 to U2, U23 to U20, U24 to U21, U25 to U22, U26 to U23, U51 to U24, U54 to U25, U28 to U26, U29 to U27, U30 to U28, U31 to U29, U5 to U3, U32 to U30, U33 to U31, U36 to U32, U37 to U33, U38 to U34, U39 to U35, U40 to U36, U41 to U37, U19 to U38, U44 to U39, U6 to U4, U45 to U40, U46 to U41, U47 to U42, U48 to U43, U34 to U44, U35 to U45, U1 to U46, U50 to U47, U49 to U48, U42 to U49, U7 to U5, U52 to U50, U53 to U51, U8 to U6, U2 to U7, U9 to U8, U10 to U9
Connections:
- net A0_1 is gone; now on net GND: U47.21 (A0), U48.15 (A0)
- net A0_2 is gone; now on net +3V3: R146.1, U50.21 (A0), U51.15 (A0)
- net A1_1 is gone; now on net GND: U47.2 (A1), U48.16 (A1)
- net A1_2 is gone; now on net GND: U50.2 (A1), U51.16 (A1)
- net A2_1 is gone; now on net GND: U47.3 (A2), U48.17 (A2)
- net A2_2 is gone; now on net GND: U50.3 (A2), U51.17 (A2)
- net Earth is gone; now on net GND: J6.1 (Pin_1), J6.3 (Pin_3), L3.2
- net +24V: now also SW2.5, SW2.7
- net +3V3: now also C42.1, C53.1, C56.1, C7.2, R10.2, R100.2, R101.2, R102.2, R103.2, R104.2, R105.2, R106.2, R107.2, R108.2, R11.2, R12.2, R120.2, R121.2, R122.2, R123.2, R124.2, R125.2, R126.2, R127.2, R128.2, R129.2, R13.2, R14.2, R140.1, R147.1, R16.2, R17.2, R18.2, R19.2, R20.2, R21.2, R33.2, R34.2, R35.2, R36.2, R37.2, R38.2, R40.2, R41.2, R42.2, R43.2, R44.2, R45.2, R54.2, R55.2, R56.2, R57.2, R58.2, R59.2, R60.2, R61.2, R62.2, R63.2, R64.2, R65.2, R75.2, R76.2, R77.2, R78.2, R79.2, R80.2, R81.2, R82.2, R83.2, R84.2, R85.2, R86.2, R9.2, R97.2, R98.2, R99.2, U38.16 (VCC), U47.24 (VDD), U48.9 (VDD), U50.24 (VDD), U51.9 (VDD), U8.5 (VS), C57.1, D34.2, D41.2, R136.1, R32.1, R39.1, U52.5 (VDD), U52.7 (A1)
- net +5V: now also BZ1.1 (-), D9.1 (K); no longer C42.1, C53.1, C56.1, C7.2, R10.2, R100.2, R101.2, R102.2, R103.2, R104.2, R105.2, R106.2, R107.2, R108.2, R11.2, R12.2, R120.2, R121.2, R122.2, R123.2, R124.2, R125.2, R126.2, R127.2, R128.2, R129.2, R13.2, R14.2, R140.1, R147.1, R16.2, R17.2, R18.2, R19.2, R20.2, R21.2, R33.2, R34.2, R35.2, R36.2, R37.2, R38.2, R40.2, R41.2, R42.2, R43.2, R44.2, R45.2, R54.2, R55.2, R56.2, R57.2, R58.2, R59.2, R60.2, R61.2, R62.2, R63.2, R64.2, R65.2, R75.2, R76.2, R77.2, R78.2, R79.2, R80.2, R81.2, R82.2, R83.2, R84.2, R85.2, R86.2, R9.2, R97.2, R98.2, R99.2, U38.16 (VCC), U47.24 (VDD), U48.9 (VDD), U50.24 (VDD), U51.9 (VDD), U8.5 (VS)
- net +5V_USB: now also C35.1, D33.1 (A1), F3.2; no longer J2.A4 (VBUS), J2.A9 (VBUS), J2.B4 (VBUS), J2.B9 (VBUS)
- net A1: now also R111.1
- net CAN_L: now also R143.1
- net EX_IO12: now also R1.1; no longer D29.1 (K), R77.1, U28.4
- net GND: now also U47.11 (P07), U47.20 (P17), U48.28 (GPA7), U48.8 (GPB7), U50.11 (P07), U50.20 (P17), U51.28 (GPA7), U51.8 (GPB7), C35.2, C43.2, C45.2, C57.2, D33.2 (A2), D34.1, D41.1, Q1.3 (C), R1.2, R112.2, R22.2, R8.2, R96.2, SW2.6, SW2.8, U52.15 (VSS), U52.6 (A0), U52.9 (A2); no longer R146.2
- net GNDA: now also R148.2, SW2.2
- net GNDS: now also U15.4 (ON/OFF)
- net I2C_SCL_HV: no longer U47.22 (SCL), U48.12 (SCK), U50.22 (SCL), U51.12 (SCK), U8.4 (SCL)
- net I2C_SDA_HV: no longer U47.23 (SDA), U48.13 (SDA), U50.23 (SDA), U51.13 (SDA), U8.3 (SDA)
- net MCP_10: now also U47.15 (P12), U48.3 (GPB2); no longer U47.14 (P11), U48.2 (GPB1)
- net MCP_11: now also U47.16 (P13), U48.4 (GPB3); no longer U47.15 (P12), U48.3 (GPB2)
- net MCP_12: now also U47.17 (P14), U48.5 (GPB4); no longer U47.16 (P13), U48.4 (GPB3)
- net MCP_13: now also U47.18 (P15), U48.6 (GPB5); no longer U47.17 (P14), U48.5 (GPB4)
- net MCP_14: now also U47.19 (P16), U48.7 (GPB6); no longer U47.18 (P15), U48.6 (GPB5)
- net MCP_15: now also U50.10 (P06), U51.27 (GPA6); no longer U47.19 (P16), U48.7 (GPB6)
- net MCP_16: now also U50.9 (P05), U51.26 (GPA5); no longer U47.20 (P17), U48.8 (GPB7)
- net MCP_17: now also U50.8 (P04), U51.25 (GPA4); no longer U50.11 (P07), U51.28 (GPA7)
- net MCP_18: now also U50.7 (P03), U51.24 (GPA3); no longer U50.10 (P06), U51.27 (GPA6)
- net MCP_19: now also U50.6 (P02), U51.23 (GPA2); no longer U50.9 (P05), U51.26 (GPA5)
- net MCP_20: now also U50.5 (P01), U51.22 (GPA1); no longer U50.8 (P04), U51.25 (GPA4)
- net MCP_21: now also U50.4 (P00), U51.21 (GPA0); no longer U50.7 (P03), U51.24 (GPA3)
- net MCP_22: now also U50.13 (P10), U51.1 (GPB0); no longer U50.6 (P02), U51.23 (GPA2)
- net MCP_23: now also U50.14 (P11), U51.2 (GPB1); no longer U50.5 (P01), U51.22 (GPA1)
- net MCP_24: now also U50.15 (P12), U51.3 (GPB2); no longer U50.4 (P00), U51.21 (GPA0)
- net MCP_25: now also U50.16 (P13), U51.4 (GPB3); no longer U50.13 (P10), U51.1 (GPB0)
- net MCP_26: now also U50.17 (P14), U51.5 (GPB4); no longer U50.14 (P11), U51.2 (GPB1)
- net MCP_27: now also U50.18 (P15), U51.6 (GPB5); no longer U50.15 (P12), U51.3 (GPB2)
- net MCP_28: now also U50.19 (P16), U51.7 (GPB6); no longer U50.16 (P13), U51.4 (GPB3)
- net MCP_8: now also U47.13 (P10), U48.1 (GPB0); no longer U47.11 (P07), U48.28 (GPA7)
- net MCP_9: now also U47.14 (P11), U48.2 (GPB1); no longer U47.13 (P10), U48.1 (GPB0)
- net USER_SWITCH: now also U52.20 (P7); no longer U7.11 (IO4)
- net VDD: now also R149.2, SW2.4
- net at Y1.1: now also U45.2 (X2); no longer U45.1 (X1)
- net at Y1.2: now also U45.1 (X1); no longer U45.2 (X2)
- net at U38.5 (UD+): now also J2.A6 (D+), J2.B6 (D+)
- net at U38.6 (UD-): now also J2.A7 (D-), J2.B7 (D-)
- net 1-WIRE renamed 1-WIRE_OUT
- net 1-WIRE_OUT: now also R132.2; no longer U7.18 (IO32)
- net A0 renamed A2
- net A2: now also R95.1
- net EX_IO17 renamed PCF_6
- net PCF_6: now also U52.17 (P5); no longer U7.21 (IO17)
- net EX_IO2 renamed BUZZER
- net BUZZER: now also R15.2, R8.1; no longer J10.5 (Pin_5)
- net EX_IO33 renamed PCF_5
- net PCF_5: now also U52.16 (P4); no longer U7.19 (IO33)
- net EX_IO36 renamed INA0
- net INA0: now also C43.1, D34.3, R95.2, R96.1
- net EX_IO39 renamed INA1
- net INA1: now also C45.1, D41.3, R111.2, R112.1
- net GPIO12_OUT renamed PCF_7_OUT
- net GPIO17_OUT renamed PCF_6_OUT
- net GPIO33_OUT renamed PCF_5_OUT
- net I2C_SCL renamed I2C_SCL_A
- net I2C_SCL_A: now also U47.22 (SCL), U48.12 (SCK), U50.22 (SCL), U51.12 (SCK), U8.4 (SCL), U52.2 (SCL); no longer I2C1.3 (Pin_3), J6.8 (Pin_8), U49.2 (LX)
- net I2C_SDA renamed I2C_SDA_A
- net I2C_SDA_A: now also U47.23 (SDA), U48.13 (SDA), U50.23 (SDA), U51.13 (SDA), U8.3 (SDA), U52.4 (SDA); no longer I2C1.4 (Pin_4), J6.7 (Pin_7), U49.3 (SX)
- net MCP_29 renamed PCF_1
- net PCF_1: now also U52.10 (P0); no longer U50.17 (P14), U51.5 (GPB4)
- net MCP_29_OUT renamed PCF_1_OUT
- net MCP_30 renamed PCF_2
- net PCF_2: now also U52.11 (P1); no longer U50.18 (P15), U51.6 (GPB5)
- net MCP_30_OUT renamed PCF_2_OUT
- net MCP_31 renamed PCF_3
- net PCF_3: now also U52.12 (P2); no longer U50.19 (P16), U51.7 (GPB6)
- net MCP_31_OUT renamed PCF_3_OUT
- net MCP_32 renamed PCF_4
- net PCF_4: now also U52.14 (P3); no longer U50.20 (P17), U51.8 (GPB7)
- net MCP_32_OUT renamed PCF_4_OUT
- new net: Q1.1 (B), R15.1, R22.1
- new net: BZ1.2 (+), D9.2 (A), Q1.2 (E)
- new net: R149.1, SW2.1
- new net: R148.1, SW2.3
- new net: R146.2, U52.1 (~{INT})
- new net: F3.1, J2.A4 (VBUS), J2.A9 (VBUS), J2.B4 (VBUS), J2.B9 (VBUS)
- new net DAT_WIRE_1: R132.1, U7.18 (IO32)
- new net DAT_WIRE_2: R133.1, U7.11 (IO4)
- new net I2C_SCL_B: I2C1.3 (Pin_3), J6.8 (Pin_8), R32.2, U49.2 (LX), U7.19 (IO33)
- new net I2C_SDA_B: I2C1.4 (Pin_4), J6.7 (Pin_7), R39.2, U49.3 (SX), U7.21 (IO17)
- new net PCF_7: D29.1 (K), R77.1, U28.4, U52.19 (P6)
- new net TEMP: J10.5 (Pin_5), R133.2, R136.2
Other:
- note added: "0x20"
- note added: "0x21"
- note added: "0x22"
- note added: "AUTO PSU Switch"
- note added: "I2C_A"
- note added: "MCP23017"
- note added: "PCF8574"
- note added: "PCF8575TS"
- note removed: "ADC"
- note removed: "Input Board v0.4 ESP"
- note removed: "MCP23017 and PCF8575"
- note removed: "Manual PSU Switch"
- note removed: "PINOUT"
- note removed: "WT32- ETH01"
- note removed: "address: 0x26"
- note removed: "address: 0x27"
- title: Input Board ESP -> (none)
- moved on the sheet: BT1, C1, C10, C11, C12, C13, C14, C15, C16, C17, C18, C19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
