File: boneIO - input WT32.kicad_sch (KiCad schematic)
At the start: 340 parts, among them J1 POWER, J10 P6, J11 P7, J2 GT-USB-7010AN, J3 UART, J4 P1, J5 P2, J6 Conn_02x04_Odd_Even, J7 P4, J8 P3, J9 P5, Q1 BC817, Q2 AO3401A, Q3 BC817, Q4 BC817, SW1 USER_SWITCH, SW2 SW_DIP_x04, U1 EL357N, U10 EL357N, U11 EL357N, U12 EL357N, U13 EL357N, U14 EL357N, U15 XL1509-5, U16 RS485, U17 EL357N, U18 EL357N, U19 EL357N, U2 EL357N, U20 EL357N, U21 EL357N, U22 EL357N, U23 RT9013-33GB, U24 SN74LVC1G3157, U25 SN74LVC1G3157, U26 EL357N, U27 EL357N, U28 EL357N, U29 EL357N, U3 EL357N, U30 EL357N, U31 EL357N, U32 EL357N, U33 EL357N, U34 EL357N, U35 EL357N, U36 EL357N, U37 EL357N, U38 CH340C, U39 EL357N, U4 EL357N, U40 EL357N, U41 EL357N, U42 EL357N, U43 EL357N, U44 2N7002DW/BSS138PS, U45 DS1307Z+, U46 SN65HVD230, U47 PCF8575, U48 MCP23017_SS, U49 PCA9515, U5 EL357N, U50 PCF8575, U51 MCP23017_SS, U52 PCF8574TS, U6 EL357N, U7 WT32-ETH01, U8 INA219AxD, U9 EL357N, Y1 32,788 MHz

Commit message: v0.6.1
Parts:
- removed D10: SMBJ5.0A, Diode_SMD:D_SMB, symbol Diode:SM6T18A
- removed D34, D41: BAT54S, Package_TO_SOT_SMD:SOT-23, symbol Diode:BAT54S
- removed R142: 0k, Resistor_SMD:R_0603_1608Metric, symbol Device:R
- added C58: 100n, Capacitor_SMD:C_0603_1608Metric, symbol Device:C
- added D10: SM712_SOT23, Package_TO_SOT_SMD:SOT-23, symbol Diode:SM712_SOT23
- added F4: JK-mSMD010-60, Fuse:Fuse_1812_4532Metric, symbol Device:Fuse
- added L4: BLM21PG121SN1D, Inductor_SMD:L_0805_2012Metric, symbol Device:L_Small
- added Q5: BC807, Package_TO_SOT_SMD:SOT-23, symbol Transistor_BJT:BC807
- added R142: 120R, Resistor_SMD:R_0805_2012Metric, symbol ESP32-EVB_Rev_I:R
- added R152: 30k, Resistor_SMD:R_0603_1608Metric, symbol Device:R
- added R153: 4.7k, Resistor_SMD:R_0603_1608Metric, symbol Device:R
- added U53: MAX485E, Package_SO:SOIC-8_3.9x4.9mm_P1.27mm, symbol Interface_UART:MAX485E
- BT1: footprint Battery:Battery_Panasonic_CR1220-VCN_Vertical_CircularHoles -> CR2032:MPD_BC501SM-TR
- C16: value 100n -> 10p
- C26: value 470p -> 100n; JLCPCB C107149 -> (none)
- F2: value 6V 500mA -> JK-mSMD010-60; footprint Fuse:Fuse_1206_3216Metric -> Fuse:Fuse_1812_4532Metric; JLCPCB (none) -> C1884489
- L1: footprint Inductor_SMD:L_7.3x7.3_H4.5 -> Inductor_SMD:L_Bourns_SRN8040TA
- R111: value 30k -> 5.1k
- R112, R96: value 4.7k -> 10k
- R136, R67: JLCPCB C238881 -> (none)
- R141: value 0k -> 4.7k; JLCPCB C269704 -> (none)
- R148, R149: value 330R -> 100k
- R150, R151: value 10k -> 4.7k
- R24: value 0k_NC -> 4.7k; footprint Resistor_SMD:R_0805_2012Metric -> Resistor_SMD:R_0603_1608Metric
- R95: value 30k -> 20k
- U24, U25: footprint Package_TO_SOT_SMD:SOT-23-6 -> Package_TO_SOT_SMD:SOT-363_SC-70-6
Connections:
- net EX_IO12 is gone; now on net DAT_WIRE_2: R1.1, U7.9 (IO12)
- net +3V3: now also J10.8 (Pin_8), R135.1, C58.1, Q5.2 (E), U53.8 (VCC); no longer J10.4 (Pin_4), R24.2
- net +5V: now also U7.25 (5V); no longer F2.2, J10.8 (Pin_8), R135.1
- net +5V_USB: no longer R67.1
- net A+_OUT: now also F4.2
- net A1: now also J10.4 (Pin_4); no longer J10.3 (Pin_3)
- net A2: now also J10.3 (Pin_3); no longer J10.2 (Pin_2)
- net B-_OUT: now also F2.2
- net CAN-RX: now also U7.11 (IO4); no longer R141.2, U7.10 (IO35)
- net CAN_L: no longer R141.1
- net DAT_WIRE_2: no longer U7.11 (IO4)
- net GND: now also R141.2, C58.2, L4.1, R153.2, U53.5 (GND)
- net GND_RS485: now also D10.3 (common), L4.2
- net RS485_RXD0: now also U53.1 (RO)
- net RS485_TXD0: now also R24.2, U53.4 (DI)
- net at C26.1: now also R67.1, Q5.3 (C), U53.2 (~{RE}), U53.3 (DE); no longer U23.4 (BP)
- net at Y1.1: now also U45.1 (X1); no longer U45.2 (X2)
- net at Y1.2: now also U45.2 (X2); no longer U45.1 (X1)
- net TEMP renamed GPIO
- net GPIO: no longer R136.2
- new net: D10.1 (A1), F4.1, R136.2, R142.1, U53.6 (A)
- new net: D10.2 (A2), F2.1, R141.1, R142.2, U53.7 (B)
- new net: Q5.1 (B), R24.1
- new net A3: J10.2 (Pin_2), R152.1
- new net INA2: C16.1, R152.2, R153.1, U7.10 (IO35)
- now unconnected: U7.16 (3V3), U7.23 (3V3)
- no-connect marks 13 -> 16
Other:
- note added: "INPUT BOARD ESP v0.6.1"
- note added: "PCU"
- note removed: "1-WIRE"
- note removed: "After connecting the USB, the pins are set to programming, after disconnecting the USB, the pins are set to RS485"
- note removed: "BUZZER"
- note removed: "EXPANDERS"
- note removed: "INA219"
- note removed: "INPUT BOARD ESP v0.5"
- note removed: "OR"
- note removed: "PINOUT"
- note removed: "PROCESOR"
- note removed: "address: 0x40"
- note removed: "address: 0x68"
- moved on the sheet: BT1, BZ1, C1, C10, C11, C12, C13, C14, C15, C17, C18, C19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

Commit message: corrected PCB schematic
Parts:
- R148, R149: value 100k -> 330R
- U1, U10, U11, U12, U13, U14, U17, U18, U19, U2, U20, U21, U22, U26, U27, U28, U29, U3, U30, U31, U32, U33, U34, U35, U36, U37, U39, U4, U40, U41, U42, U43, U5, U6, U9: value EL357N -> EL354N
Changed lines of the file:
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@@
       (effects (font (size 1.27 1.27)))
     )
-    (property "Value" "EL357N" (at 72.39 409.9814 0)
+    (property "Value" "EL354N" (at 72.39 409.9814 0)
       (effects (font (size 1.27 1.27)))
     )
@@
       (effects (font (size 1.27 1.27)))
     )
-    (property "Value" "EL357N" (at 151.13 486.1814 0)
+    (property "Value" "EL354N" (at 151.13 486.1814 0)
       (effects (font (size 1.27 1.27)))
     )
@@
       (effects (font (size 1.27 1.27)))
     )
-    (property "Value" "EL357N" (at 232.41 294.4114 0)
+    (property "Value" "EL354N" (at 232.41 294.4114 0)
       (effects (font (size 1.27 1.27)))
     )
@@
       (effects (font (size 1.27 1.27)))
     )
-    (property "Value" "EL357N" (at 480.06 294.4114 0)
+    (property "Value" "EL354N" (at 480.06 294.4114 0)
       (effects (font (size 1.27 1.27)))
     )
@@
       (effects (font (size 1.27 1.27)))
     )
-    (property "Value" "EL357N" (at 72.39 371.8814 0)
+    (property "Value" "EL354N" (at 72.39 371.8814 0)
       (effects (font (size 1.27 1.27)))
     )
@@
       (effects (font (size 1.27 1.27)))
     )
-    (property "Value" "EL357N" (at 480.06 371.8814 0)
+    (property "Value" "EL354N" (at 480.06 371.8814 0)
       (effects (font (size 1.27 1.27)))
     )
@@
       (effects (font (size 1.27 1.27)))
     )
-    (property "Value" "EL357N" (at 232.41 448.0814 0)
+    (property "Value" "EL354N" (at 232.41 448.0814 0)
       (effects (font (size 1.27 1.27)))
     )
@@
       (effects (font (size 1.27 1.27)))
     )
-    (property "Value" "EL357N" (at 72.39 333.7814 0)
+    (property "Value" "EL354N" (at 72.39 333.7814 0)
       (effects (font (size 1.27 1.27)))
     )
@@
       (effects (font (size 1.27 1.27)))
     )
-    (property "Value" "EL357N" (at 232.41 333.7814 0)
+    (property "Value" "EL354N" (at 232.41 333.7814 0)
       (effects (font (size 1.27 1.27)))
     )
@@
       (effects (font (size 1.27 1.27)) (justify left))
     )
-    (property "Value" "100k" (at 523.24 217.17 90)
+    (property "Value" "330R" (at 523.24 217.17 90)
       (effects (font (size 1.27 1.27)) (justify left))
     )
@@
       (effects (font (size 1.27 1.27)))
     )
-    (property "Value" "EL357N" (at 151.13 333.7814 0)
+    (property "Value" "EL354N" (at 151.13 333.7814 0)
       (effects (font (size 1.27 1.27)))
     )
@@
       (effects (font (size 1.27 1.27)))
     )
-    (property "Value" "EL357N" (at 151.13 448.0814 0)
+    (property "Value" "EL354N" (at 151.13 448.0814 0)
       (effects (font (size 1.27 1.27)))
     )
@@
       (effects (font (size 1.27 1.27)) (justify left))
     )
-    (property "Value" "100k" (at 523.24 212.09 90)
+    (property "Value" "330R" (at 523.24 212.09 90)
       (effects (font (size 1.27 1.27)) (justify left))
     )
@@
       (effects (font (size 1.27 1.27)))
     )
-    (property "Value" "EL357N" (at 314.96 373.1514 0)
+    (property "Value" "EL354N" (at 314.96 373.1514 0)
       (effects (font (size 1.27 1.27)))
     )
@@
       (effects (font (size 1.27 1.27)))
     )
-    (property "Value" "EL357N" (at 397.51 333.7814 0)
+    (property "Value" "EL354N" (at 397.51 333.7814 0)
       (effects (font (size 1.27 1.27)))
     )
@@
       (effects (font (size 1.27 1.27)))
     )
-    (property "Value" "EL357N" (at 397.51 448.0814 0)
+    (property "Value" "EL354N" (at 397.51 448.0814 0)
       (effects (font (size 1.27 1.27)))
     )
@@
       (effects (font (size 1.27 1.27)))
     )
-    (property "Value" "EL357N" (at 397.51 486.1814 0)
+    (property "Value" "EL354N" (at 397.51 486.1814 0)
       (effects (font (size 1.27 1.27)))
     )
@@
       (effects (font (size 1.27 1.27)))
     )
-    (property "Value" "EL357N" (at 480.06 451.8914 0)
+    (property "Value" "EL354N" (at 480.06 451.8914 0)
       (effects (font (size 1.27 1.27)))
     )
@@
       (effects (font (size 1.27 1.27)))
     )
-    (property "Value" "EL357N" (at 151.13 294.4114 0)
+    (property "Value" "EL354N" (at 151.13 294.4114 0)
       (effects (font (size 1.27 1.27)))
     )
@@
       (effects (font (size 1.27 1.27)))
     )
-    (property "Value" "EL357N" (at 314.96 333.7814 0)
+    (property "Value" "EL354N" (at 314.96 333.7814 0)
       (effects (font (size 1.27 1.27)))
     )
@@
       (effects (font (size 1.27 1.27)))
     )
-    (property "Value" "EL357N" (at 72.39 294.4114 0)
+    (property "Value" "EL354N" (at 72.39 294.4114 0)
       (effects (font (size 1.27 1.27)))
     )
@@
       (effects (font (size 1.27 1.27)))
     )
-    (property "Value" "EL357N" (at 151.13 371.8814 0)
+    (property "Value" "EL354N" (at 151.13 371.8814 0)
       (effects (font (size 1.27 1.27)))
     )
@@
       (effects (font (size 1.27 1.27)))
     )
-    (property "Value" "EL357N" (at 314.96 453.1614 0)
+    (property "Value" "EL354N" (at 314.96 453.1614 0)
       (effects (font (size 1.27 1.27)))
     )
@@
       (effects (font (size 1.27 1.27)))
     )
-    (property "Value" "EL357N" (at 232.41 486.1814 0)
+    (property "Value" "EL354N" (at 232.41 486.1814 0)
       (effects (font (size 1.27 1.27)))
     )
@@
       (effects (font (size 1.27 1.27)))
     )
-    (property "Value" "EL357N" (at 397.51 409.9814 0)
+    (property "Value" "EL354N" (at 397.51 409.9814 0)
       (effects (font (size 1.27 1.27)))
     )
@@
       (effects (font (size 1.27 1.27)))
     )
-    (property "Value" "EL357N" (at 72.39 486.1814 0)
+    (property "Value" "EL354N" (at 72.39 486.1814 0)
       (effects (font (size 1.27 1.27)))
     )
@@
       (effects (font (size 1.27 1.27)))
     )
-    (property "Value" "EL357N" (at 314.96 412.5214 0)
+    (property "Value" "EL354N" (at 314.96 412.5214 0)
       (effects (font (size 1.27 1.27)))
     )
@@
       (effects (font (size 1.27 1.27)))
     )
-    (property "Value" "EL357N" (at 314.96 294.4114 0)
+    (property "Value" "EL354N" (at 314.96 294.4114 0)
       (effects (font (size 1.27 1.27)))
     )
@@
       (effects (font (size 1.27 1.27)))
     )
-    (property "Value" "EL357N" (at 72.39 448.0814 0)
+    (property "Value" "EL354N" (at 72.39 448.0814 0)
       (effects (font (size 1.27 1.27)))
     )
@@
       (effects (font (size 1.27 1.27)))
     )
-    (property "Value" "EL357N" (at 232.41 371.8814 0)
+    (property "Value" "EL354N" (at 232.41 371.8814 0)
       (effects (font (size 1.27 1.27)))
     )
@@
       (effects (font (size 1.27 1.27)))
     )
-    (property "Value" "EL357N" (at 480.06 333.7814 0)
+    (property "Value" "EL354N" (at 480.06 333.7814 0)
       (effects (font (size 1.27 1.27)))
     )
@@
       (effects (font (size 1.27 1.27)))
     )
-    (property "Value" "EL357N" (at 151.13 409.9814 0)
+    (property "Value" "EL354N" (at 151.13 409.9814 0)
       (effects (font (size 1.27 1.27)))
     )
@@
       (effects (font (size 1.27 1.27)))
     )
-    (property "Value" "EL357N" (at 480.06 409.9814 0)
+    (property "Value" "EL354N" (at 480.06 409.9814 0)
       (effects (font (size 1.27 1.27)))
     )
@@
       (effects (font (size 1.27 1.27)))
     )
-    (property "Value" "EL357N" (at 314.96 493.8014 0)
+    (property "Value" "EL354N" (at 314.96 493.8014 0)
       (effects (font (size 1.27 1.27)))
     )
@@
       (effects (font (size 1.27 1.27)))
     )
-    (property "Value" "EL357N" (at 397.51 371.8814 0)
+    (property "Value" "EL354N" (at 397.51 371.8814 0)
       (effects (font (size 1.27 1.27)))
     )
@@
       (effects (font (size 1.27 1.27)))
     )
-    (property "Value" "EL357N" (at 232.41 409.9814 0)
+    (property "Value" "EL354N" (at 232.41 409.9814 0)
       (effects (font (size 1.27 1.27)))
     )
@@
       (effects (font (size 1.27 1.27)))
     )
-    (property "Value" "EL357N" (at 397.51 294.4114 0)
+    (property "Value" "EL354N" (at 397.51 294.4114 0)
       (effects (font (size 1.27 1.27)))
     )

Commit message: v0.6.4
Changes made:
- Replacement of stabilizer with ST1S12XX inverters
- Improved 24V power supply paths
- Replacement of input power switch
- Elimination of automatic programmer-rs485 flip-flop
Parts:
- removed R148, R149: 330R, Resistor_SMD:R_1206_3216Metric, symbol Device:R
- removed R53: 4.7k, Resistor_SMD:R_0603_1608Metric, symbol Device:R
- removed SW2: SW_DIP_x04, Button_Switch_THT:SW_DIP_SPSTx04_Piano_10.8x11.72mm_W7.62mm_P2.54mm, symbol Switch:SW_DIP_x04
- removed U16: RS485, rs485:RS485_moduleTTL, symbol RS485:RS485_module
- removed U23: RT9013-33GB, Package_TO_SOT_SMD:SOT-23-5, symbol Reference_Voltage:RT9013-33GB
- removed U24, U25: SN74LVC1G3157, Package_TO_SOT_SMD:SOT-363_SC-70-6, symbol SN74LVC1G3157:SN74LVC1G3157
- added L5: 2.2uH, Inductor_SMD:L_Bourns-SRN4018, symbol Device:L_Small
- added R154: 100k, Resistor_SMD:R_0603_1608Metric, symbol Device:R
- added R155: 68k_1%, Resistor_SMD:R_0603_1608Metric, symbol Device:R
- added R156: 15K_1%, Resistor_SMD:R_0603_1608Metric, symbol Device:R
- added U16: ST1S12XX, Package_TO_SOT_SMD:TSOT-23-5, symbol Regulator_Switching:ST1S12XX
- added U23: SK-23D07, switch:SK-23D07, symbol Switch:SK-23D07
- D18, D26: footprint LED_SMD:LED_0805_2012Metric -> LED_SMD:LED_0603_1608Metric
Connections:
- net CH_RXD is gone; now on net IO3_RXD0: U38.2 (TXD)
- net CH_TXD is gone; now on net IO1_TXD0: U38.3 (RXD)
- net RS485_RXD0 is gone; now on net IO3_RXD0: U53.1 (RO)
- net RS485_TXD0 is gone; now on net IO1_TXD0: R24.2, U53.4 (DI)
- net +24V: now also U23.4, U23.5
- net +3V3: now also L5.2, R155.1
- net +5V: now also R154.2, U16.4 (V_{IN})
- net GND: now also Q1.2 (E), R156.2, U16.2 (GND), U23.1, U23.8, U23.9 (GND); no longer Q1.3 (C)
- net GNDA: now also U23.6
- net VDD: now also U23.2
- net at BZ1.2 (+), D9.2 (A): now also Q1.3 (C); no longer Q1.2 (E)
- new net: R155.2, R156.1, U16.5 (FB/V_{O})
- new net: R154.1, U16.1 (EN)
- new net: L5.1, U16.3 (SW)
- no-connect marks 16 -> 17
Other:
- note added: "INPUT BOARD ESP v0.6.3"
- note added: "MANUAL PSU Switch"
- note removed: "AUTO PSU Switch"
- note removed: "Automatic UART switching"
- note removed: "INPUT BOARD ESP v0.6.1"
- moved on the sheet: C27, D26, R66

Commit message: input_board_ESP_v0.7.0
Changes:
- replacement of 5V DC converter with TPS54202DDC
- replacement of 3.3V DC converter with TLV62569DBV
- removal of RTC zagar
- replacement of programmer for CH340K
- Merging two i2c buses into one
- connecting rs485 to gpio pins 14 and 15
Parts:
- removed BT1: Battery, CR2032:MPD_BC501SM-TR, symbol Device:Battery
- removed C17, C42, C44, C51: 100n, Capacitor_SMD:C_0603_1608Metric, symbol Device:C
- removed C18, C25, C27: 10u, Capacitor_SMD:C_1206_3216Metric, symbol Device:C
- removed D11: SS34, Diode_SMD:D_SMA, symbol Device:D_ALT
- removed L1: 68uH, Inductor_SMD:L_Bourns_SRN8040TA, symbol Device:L_Small
- removed L4: BLM21PG121SN1D, Inductor_SMD:L_0805_2012Metric, symbol Device:L_Small
- removed L5: 2.2uH, Inductor_SMD:L_Bourns-SRN4018, symbol Device:L_Small
- removed Q3, Q4: BC817, Package_TO_SOT_SMD:SOT-23, symbol Transistor_BJT:BC817
- removed R109, R110, R138: 10k, Resistor_SMD:R_0603_1608Metric, symbol Device:R
- removed R130, R131, R134, R137: 4.7k, Resistor_SMD:R_0603_1608Metric, symbol Device:R
- removed R154: 100k, Resistor_SMD:R_0603_1608Metric, symbol Device:R
- removed R155: 68k_1%, Resistor_SMD:R_0603_1608Metric, symbol Device:R
- removed R156: 15K_1%, Resistor_SMD:R_0603_1608Metric, symbol Device:R
- removed U15: XL1509-5, Package_SO:SOP-8_3.9x4.9mm_P1.27mm, symbol Power_Management:XL1509-5
- removed U16: ST1S12XX, Package_TO_SOT_SMD:TSOT-23-5, symbol Regulator_Switching:ST1S12XX
- removed U38: CH340C, Package_SO:SOIC-16_3.9x9.9mm_P1.27mm, symbol Interface_USB:CH340C
- removed U44: 2N7002DW/BSS138PS, Package_TO_SOT_SMD:SOT-363_SC-70-6, symbol Transistor_FET:2N7002DW
- removed U45: DS1307Z+, Package_SO:SOIC-8_3.9x4.9mm_P1.27mm, symbol Timer_RTC:DS1307Z+
- removed Y1: 32,788 MHz, Crystal:Crystal_C26-LF_D2.1mm_L6.5mm_Horizontal, symbol Device:Crystal
- added C1: 4.7uF/C0805, Capacitor_SMD:C_0805_2012Metric, symbol Device:C
- added C1: 10uF/C0805, Capacitor_SMD:C_0603_1608Metric, symbol Device:C
- added C10: 47uF/C1210, Capacitor_SMD:C_1210_3225Metric, symbol Device:C
- added C2, C8: 100nF/C603, Capacitor_SMD:C_0603_1608Metric, symbol Device:C
- added C2: 22uF/C1206, Capacitor_SMD:C_1206_3216Metric, symbol Device:C
- added C3: 6.8pF/C0603, Capacitor_SMD:C_0603_1608Metric, symbol Device:C
- added C6: 2.2uF/C0805, Capacitor_SMD:C_0805_2012Metric, symbol Device:C
- added C7: 1uF/C0805, Capacitor_SMD:C_0805_2012Metric, symbol Device:C
- added C9: 68pF/C0603, Capacitor_SMD:C_0603_1608Metric, symbol Device:C
- added L2: FNR6045S150MT/SRN6028, Inductor_SMD:L_Bourns-SRN6028, symbol Device:L_Small
- added L2: CY43-2.2UH/SRN4018, Inductor_SMD:L_Bourns-SRN4018, symbol Device:L_Small
- added Q1, Q2: BC817/SOT-23, Package_TO_SOT_SMD:SOT-23, symbol Transistor_BJT:BC817
- added R1: 210k/R0603, Resistor_SMD:R_0603_1608Metric, symbol Mazda_EMU_v2-rescue:R-Device-Mazda_EMU_v1-rescue
- added R2: 47k/R0603, Resistor_SMD:R_0603_1608Metric, symbol Mazda_EMU_v2-rescue:R-Device-Mazda_EMU_v1-rescue
- added R3: 100k/R0603, Resistor_SMD:R_0603_1608Metric, symbol Mazda_EMU_v2-rescue:R-Device-Mazda_EMU_v1-rescue
- added R4: 13.7k/R0603, Resistor_SMD:R_0603_1608Metric, symbol Mazda_EMU_v2-rescue:R-Device-Mazda_EMU_v1-rescue
- added R5, R6: 4.7k/R0603, Resistor_SMD:R_0603_1608Metric, symbol Device:R
- added U1: TLV62569DBV/SOT23-5, Package_TO_SOT_SMD:SOT-23-5, symbol Regulator_Switching:TLV62569DBV
- added U1: CH340K/SSOP-10, Package_SO:SSOP-10_3.9x4.9mm_P1.00mm, symbol Interface_USB:CH340K
- added U2: TPS54202DDC/SOT-23-6, Package_TO_SOT_SMD:SOT-23-6, symbol Regulator_Switching:TPS54202DDC
- BZ1: JLCPCB (none) -> C96493
- C1, C2, C3, C4, C5, C6, C7: value 100n -> 100nF/C603
- C11: renamed from C10; value 100n -> 100nF/C603
- C12: renamed from C11; value 100n -> 100nF/C603
- C13: renamed from C12; value 100n -> 100nF/C603
- C14: renamed from C13; value 100n -> 100nF/C603
- C15: renamed from C14; value 100n -> 100nF/C603
- C16: renamed from C15; value 100n -> 100nF/C603
- C20: renamed from C19; value 100n -> 100nF/C603
- C21: renamed from C20; value 100n -> 100nF/C603
- C22: renamed from C21; value 100n -> 100nF/C603
- C23: renamed from C22; value 100n -> 100nF/C603
- C24: renamed from C23; value 100n -> 100nF/C603
- C25: renamed from C24; value 100n -> 100nF/C603
- C30: renamed from C52; value 100n -> 100nF/C603
- C31: renamed from C28; value 100n -> 100nF/C603
- C32: renamed from C29; value 100n -> 100nF/C603
- C33: renamed from C30; value 100n -> 100nF/C603
- C34: renamed from C31; value 100n -> 100nF/C603
- C35: renamed from C32; value 100n -> 100nF/C603
- C36: renamed from C33; value 100n -> 100nF/C603
- C38: renamed from C34; value 4.7n -> 4.7n/C0603
- C39: renamed from C35; value 100n -> 100nF/C603
- C40: renamed from C55; value 100n -> 100nF/C603
- C41: renamed from C36; value 100n -> 100nF/C603
- C42: renamed from C37; value 100n -> 100nF/C603
- C43: renamed from C38; value 100n -> 100nF/C603
- C44: renamed from C39; value 100n -> 100nF/C603
- C45: renamed from C40; value 100n -> 100nF/C603
- C46: renamed from C41; value 100n -> 100nF/C603
- C49: renamed from C46; value 100n -> 100nF/C603
- C50: renamed from C47; value 100n -> 100nF/C603
- C51: renamed from C48; value 100n -> 100nF/C603
- C52: renamed from C49; value 100n -> 100nF/C603
- C53: renamed from C50; value 100n -> 100nF/C603
- C54: renamed from C53; value 100n -> 100nF/C603
- C55: renamed from C26; value 100n -> 100nF/C603
- C56: renamed from C58; value 100n -> 100nF/C603
- C57: renamed from C56; value 100n -> 100nF/C603
- C58: renamed from C57; value 100n -> 100nF/C603
- C59: renamed from C43; value 10p -> 10p/C0603
- C60: renamed from C54; value 100n -> 100nF/C603
- C61: renamed from C16; value 10p -> 10p/C0603
- C62: renamed from C45; value 10p -> 10p/C0603
- C8: value 220uF/50v -> 220uF/50v/CP8x10
- C9: value 10uF -> 10uF/C603
- D1: value SMBJ28CA -> SMBJ28CA/SMB; JLCPCB (none) -> C353369
- D10: renamed from D13; value LED -> LED_RED/L0603
- D11: renamed from D14; value LED -> LED_RED/L0603
- D12: renamed from D15; value LED -> LED_RED/L0603
- D13: renamed from D16; value LED -> LED_RED/L0603
- D14: renamed from D17; value LED -> LED_RED/L0603
- D15: renamed from D18; value LED_RED -> LED_RED/L0603
- D16: renamed from D19; value B5819W -> B5819W/SOD-123
- D17: renamed from D20; value LED -> LED_RED/L0603
- D18: renamed from D21; value LED -> LED_RED/L0603
- D19: renamed from D22; value LED -> LED_RED/L0603
- D2: value SS34 -> SS34/SMA; JLCPCB C64982 -> C8678
- D20: renamed from D23; value LED -> LED_RED/L0603
- D21: renamed from D24; value LED -> LED_RED/L0603
- D22: renamed from D25; value LED -> LED_RED/L0603
- D23: renamed from D26; value LED_RED -> LED_RED/L0603
- D24: renamed from D50; value PESD1CAN -> PESD1CAN/SOT-23
- D25: renamed from D27; value LED -> LED_RED/L0603
- D26: renamed from D28; value LED -> LED_RED/L0603
- D27: renamed from D29; value LED -> LED_RED/L0603
- D28: renamed from D30; value LED -> LED_RED/L0603
- D29: renamed from D31; value LED -> LED_RED/L0603
- D3, D4, D5, D6, D7, D8: value LED -> LED_RED/L0603
- D30: renamed from D32; value LED -> LED_RED/L0603
- D31: renamed from D33; value SMBJ5.0A -> SMBJ5.0A/SMB
- D32: renamed from D35; value LED -> LED_RED/L0603
- D33: renamed from D36; value LED -> LED_RED/L0603
- D34: renamed from D37; value LED -> LED_RED/L0603
- D35: renamed from D38; value LED -> LED_RED/L0603
- D36: renamed from D39; value LED -> LED_RED/L0603
- D37: renamed from D40; value LED -> LED_RED/L0603
- D38: renamed from D51; value PESD5V0S2BT -> PESD5V0S2BT/SOT-23
- D39: renamed from D42; value LED_GREEN -> LED_RED/L0603
- D40: renamed from D43; value LED_GREEN -> LED_GREEN/L0603
- D41: renamed from D44; value LED -> LED_RED/L0603
- D42: renamed from D45; value LED -> LED_RED/L0603
- D43: renamed from D46; value LED -> LED_RED/L0603
- D44: renamed from D47; value LED -> LED_RED/L0603
- D45: renamed from D48; value LED -> LED_RED/L0603
- D46: renamed from D9; value 1N4148 -> LL4148/MiniMELF
- D47: renamed from D10; value SM712_SOT23 -> SM712/SOT23
- D48: renamed from D49; value 1N4148 -> LL4148/MiniMELF
- D9: renamed from D12; value LED -> LED_RED/L0603
- F1: value MF-MSMF075/24-2 -> MF-MSMF110/24X-2/L1812; JLCPCB (none) -> C210835
- F2: renamed from F3; value 6V 500mA -> 6V 500mA /L1206
- F3: renamed from F2; value JK-mSMD010-60 -> JK-mSMD010-60/L1812
- F4: value JK-mSMD010-60 -> JK-mSMD010-60/L1812
- J2: value GT-USB-7010AN -> GT-USB-7010AN/USB-C
- L2, L3: value BLM21PG121SN1D -> BLM21PG121SN1D/L0805
- Q1: renamed from Q2; value AO3401A -> AO3401A/SOT-23
- Q4: renamed from Q1; value BC817 -> BC817/SOT-23
- Q5: value BC807 -> BC807/SOT-23
- R1, R10, R11, R114, R115, R116, R117, R12, R120, R121, R122, R123, R124, R13, R14, R2, R3, R4, R5, R6, R7, R8, R9: value 10k -> 10k/R0603
- R100: renamed from R98; value 10k -> 10k/R0603
- R101: renamed from R99; value 10k -> 10k/R0603
- R102: renamed from R100; value 10k -> 10k/R0603
- R103: renamed from R101; value 10k -> 10k/R0603
- R104: renamed from R102; value 10k -> 10k/R0603
- R105: renamed from R150; value 4.7k -> 4.7k/R0603/NC
- R106: renamed from R103; value 1.2k -> 1.2k/R0603
- R107: renamed from R104; value 1.2k -> 1.2k/R0603
- R108: renamed from R105; value 1.2k -> 1.2k/R0603
- R109: renamed from R106; value 1.2k -> 1.2k/R0603
- R110: renamed from R107; value 1.2k -> 1.2k/R0603
- R111: renamed from R108; value 1.2k -> 1.2k/R0603
- R112: renamed from R151; value 4.7k -> 4.7k/R0603/NC
- R113: value 4.7k -> 4.7k/R0603
- R118, R119, R125, R126, R127, R128, R129, R16, R17, R18, R19, R20, R21: value 1.2k -> 1.2k/R0603
- R132, R133: value 100R -> 100R/R0603
- R134: renamed from R135; value 4.7k -> 4.7k/R0603
- R136: renamed from R140; value 4.7k -> 4.7k/R0603
- R138: renamed from R15; value 1.2k -> 1.2k/R0603
- R139: renamed from R24; value 4.7k -> 4.7k/R0603
- R140: renamed from R22; value 10k -> 10k/R0603
- R141: renamed from R67; value 4.7k -> 4.7k/R0603
- R143: renamed from R146; value 4.7k -> 4.7k/R0603
- R144: renamed from R147; value 4.7k -> 4.7k/R0603
- R145: renamed from R136; value 4.7k -> 4.7k/R0603
- R146: renamed from R141; value 4.7k -> 4.7k/R0603
- R147: renamed from R142; value 120R -> 120R/R0603; footprint Resistor_SMD:R_0805_2012Metric -> Resistor_SMD:R_0603_1608Metric
- R148: renamed from R95; value 20k -> 20k/R0603
- R149: renamed from R96; value 10k -> 10k/R0603
- R15: renamed from R23; value 0.1R_1% -> 0.1R_1%/R2512
- R150: renamed from R152; value 30k -> 30k/R0603
- R151: renamed from R153; value 4.7k -> 4.7k/R0603
- R152: renamed from R144; value 4.7k -> 4.7k/R0603
- R153: renamed from R145; value 330R -> 330R/R0603
- R154: renamed from R111; value 5.1k -> 5.1k/R0603
- R155: renamed from R112; value 10k -> 10k/R0603
- R22: renamed from R25; value 4.7k -> 4.7k/R0603
- R23: renamed from R26; value 10k -> 10k/R0603
- R24: renamed from R27; value 10k -> 10k/R0603
- R25: renamed from R28; value 10k -> 10k/R0603
- R26: renamed from R29; value 10k -> 10k/R0603
- R27: renamed from R30; value 10k -> 10k/R0603
- R28: renamed from R31; value 10k -> 10k/R0603
- R29: renamed from R32; value 4.7k -> 4.7k/R0603
- R30: renamed from R33; value 10k -> 10k/R0603
- R31: renamed from R34; value 10k -> 10k/R0603
- R32: renamed from R35; value 10k -> 10k/R0603
- R33: renamed from R36; value 10k -> 10k/R0603
- R34: renamed from R37; value 10k -> 10k/R0603
- R35: renamed from R38; value 10k -> 10k/R0603
- R36: renamed from R39; value 4.7k -> 4.7k/R0603
- R37: renamed from R40; value 1.2k -> 1.2k/R0603
- R38: renamed from R41; value 1.2k -> 1.2k/R0603
- R39: renamed from R42; value 1.2k -> 1.2k/R0603
- R40: renamed from R43; value 1.2k -> 1.2k/R0603
- R41: renamed from R44; value 1.2k -> 1.2k/R0603
- R42: renamed from R45; value 1.2k -> 1.2k/R0603
- R45: renamed from R46; value 1.2k -> 1.2k/R0603
- R46: renamed from R47; value 10k -> 10k/R0603
- R47: renamed from R48; value 10k -> 10k/R0603
- R48: renamed from R49; value 10k -> 10k/R0603
- R49: renamed from R50; value 10k -> 10k/R0603
- R50: renamed from R51; value 10k -> 10k/R0603
- R51: renamed from R52; value 10k -> 10k/R0603
- R52: renamed from R54; value 10k -> 10k/R0603
- R53: renamed from R55; value 10k -> 10k/R0603
- R54: renamed from R56; value 10k -> 10k/R0603
- R55: renamed from R57; value 10k -> 10k/R0603
- R56: renamed from R58; value 10k -> 10k/R0603
- R57: renamed from R59; value 10k -> 10k/R0603
- R59: renamed from R60; value 1.2k -> 1.2k/R0603
- R60: renamed from R61; value 1.2k -> 1.2k/R0603
- R61: renamed from R62; value 1.2k -> 1.2k/R0603
- R62: renamed from R63; value 1.2k -> 1.2k/R0603
- R63: renamed from R64; value 1.2k -> 1.2k/R0603
- R64: renamed from R65; value 1.2k -> 1.2k/R0603
- R65: renamed from R66; value 1.2k -> 1.2k/R0603
- R68: renamed from R139; value 10k -> 10k/R0603
- R69: renamed from R68; value 10k -> 10k/R0603
- R70: renamed from R69; value 10k -> 10k/R0603
- R71: renamed from R70; value 10k -> 10k/R0603
- R72: renamed from R71; value 10k -> 10k/R0603
- R73: renamed from R72; value 10k -> 10k/R0603
- R74: renamed from R73; value 10k -> 10k/R0603
- R75: renamed from R74; value 1M -> 1M/R0603
- R76: renamed from R143; value 120R -> 120R/R0603; footprint Resistor_SMD:R_0805_2012Metric -> Resistor_SMD:R_0603_1608Metric
- R77: renamed from R75; value 10k -> 10k/R0603
- R78: renamed from R76; value 10k -> 10k/R0603
- R79: renamed from R77; value 10k -> 10k/R0603
- R80: renamed from R78; value 10k -> 10k/R0603
- R81: renamed from R79; value 10k -> 10k/R0603
- R82: renamed from R80; value 10k -> 10k/R0603
- R83: renamed from R81; value 1.2k -> 1.2k/R0603
- R84: renamed from R82; value 1.2k -> 1.2k/R0603
- R85: renamed from R83; value 1.2k -> 1.2k/R0603
- R86: renamed from R84; value 1.2k -> 1.2k/R0603
- R87: renamed from R85; value 1.2k -> 1.2k/R0603
- R88: renamed from R86; value 1.2k -> 1.2k/R0603
- R89: renamed from R87; value 5.1k -> 5.1k/R0603
- R90: renamed from R88; value 5.1k -> 5.1k/R0603
- R91: renamed from R89; value 10k -> 10k/R0603
- R92: renamed from R90; value 10k -> 10k/R0603
- R93: renamed from R91; value 10k -> 10k/R0603
- R94: renamed from R92; value 10k -> 10k/R0603
- R95: renamed from R93; value 10k -> 10k/R0603
- R96: renamed from R94; value 10k -> 10k/R0603
- R99: renamed from R97; value 10k -> 10k/R0603
- RV1: value 07D270K -> 07D270K/NC; JLCPCB C317745 -> C273545
- U10: renamed from U9; value EL354N -> EL354N/SOP-4
- U11: renamed from U10; value EL354N -> EL354N/SOP-4
- U12: renamed from U11; value EL354N -> EL354N/SOP-4
- U13: renamed from U12; value EL354N -> EL354N/SOP-4
- U14: renamed from U13; value EL354N -> EL354N/SOP-4
- U15: renamed from U14; value EL354N -> EL354N/SOP-4
- U17, U18, U19, U20, U21, U22, U39, U40, U41, U42, U43: value EL354N -> EL354N/SOP-4
- U2: renamed from U1; value EL354N -> EL354N/SOP-4
- U24: renamed from U46; value SN65HVD230 -> SN65HVD230/SO-8
- U25: renamed from U26; value EL354N -> EL354N/SOP-4
- U26: renamed from U27; value EL354N -> EL354N/SOP-4
- U27: renamed from U28; value EL354N -> EL354N/SOP-4
- U28: renamed from U29; value EL354N -> EL354N/SOP-4
- U29: renamed from U30; value EL354N -> EL354N/SOP-4
- U3: renamed from U2; value EL354N -> EL354N/SOP-4
- U30: renamed from U31; value EL354N -> EL354N/SOP-4
- U32: renamed from U49; value PCA9515 -> PCA9515/SSOP-8
- U33: renamed from U32; value EL354N -> EL354N/SOP-4
- U34: renamed from U33; value EL354N -> EL354N/SOP-4
- U35: renamed from U34; value EL354N -> EL354N/SOP-4
- U36: renamed from U35; value EL354N -> EL354N/SOP-4
- U37: renamed from U36; value EL354N -> EL354N/SOP-4
- U38: renamed from U37; value EL354N -> EL354N/SOP-4
- U4: renamed from U3; value EL354N -> EL354N/SOP-4
- U46: renamed from U47; value PCF8575 -> PCF8575/SSOP-24
- U47: renamed from U48; value MCP23017_SS -> MCP23017_SS/SSOP-28
- U48: renamed from U53; value MAX485E -> MAX485E/SO-8
- U5: renamed from U4; value EL354N -> EL354N/SOP-4
- U50: value PCF8575 -> PCF8575/SSOP-24
- U51: value MCP23017_SS -> MCP23017_SS/SSOP-28
- U52: value PCF8574TS -> PCF8574TS/SSOP-20
- U6: renamed from U5; value EL354N -> EL354N/SOP-4
- U7: renamed from U6; value EL354N -> EL354N/SOP-4
- U8: value INA219AxD -> INA219AxD/SO-8
- renumbered J7 to J10, J8 to J11, J9 to J6, J10 to J7, J6 to J8, J11 to J9, U7 to U1, U23 to U44
Connections:
- net GND_RS485 is gone; now on net GND: D47.3 (common), J9.3 (Pin_3)
- net I2C_SCL_B is gone; now on net I2C_SCL: I2C1.3 (Pin_3), J8.8 (Pin_8), R29.2, U1.19 (IO33), U32.2 (LX)
- net I2C_SDA_B is gone; now on net I2C_SDA: I2C1.4 (Pin_4), J8.7 (Pin_7), R36.2, U1.21 (IO17), U32.3 (SX)
- net +24V: now also C2.1, U2.3 (VIN)
- net +3V3: now also C1.2, C2.2, C3.2, C6.1, C7.1, L2.2, R1.2, U1.10 (V3), U1.7 (VCC)
- net +5V: now also C1.1, U1.1 (EN), U1.4 (VIN)
- net ESP_EN: now also Q1.3 (C)
- net GND: now also C1.1, C1.2, C2.1, C6.2, C7.2, R2.1, U1.11 (GND), U1.2 (GND), U1.3 (GND)
- net GNDS: now also C10.2, C2.2, R4.2, U2.1 (GND)
- net GPIO0: now also Q2.3 (C)
- net at D16.2 (A), Q1.1 (G), R45.1: now also C10.1, C9.1, L2.2, R3.1
- net UD+: now reaches J2.A6 (D+), J2.B6 (D+)
- net UD+: now also U1.1 (UD+)
- net UD-: now reaches J2.A7 (D-), J2.B7 (D-)
- net UD-: now also U1.2 (UD-)
- net I2C_SCL_A renamed I2C_SCL
- net I2C_SCL: no longer U1.7 (IO15)
- net I2C_SDA_A renamed I2C_SDA
- net I2C_SDA: no longer U1.8 (IO14)
- net IO1_TXD0 renamed CH_TXD
- net CH_TXD: now also U1.9 (RXD); no longer R139.2, U48.4 (DI)
- net IO3_RXD0 renamed CH_RXD
- net CH_RXD: now also U1.8 (TXD); no longer U48.1 (RO)
- new net: Q1.1 (B), R5.1
- new net: Q2.1 (B), R6.1
- new net: C9.2, R3.2, R4.1, U2.4 (FB)
- new net: C3.1, R1.1, R2.2, U1.5 (FB)
- new net: L2.1, U1.3 (SW)
- new net: C8.1, L2.1, U2.2 (SW)
- new net: C8.2, U2.6 (BOOT)
- new net DTR: Q2.2 (E), R5.2, U1.4 (DTR#)
- new net RS485_RXD0: U1.8 (IO14), U48.1 (RO)
- new net RS485_TXD0: R139.2, U1.7 (IO15), U48.4 (DI)
- new net RTS: Q1.2 (E), R6.2, U1.6 (RTS#)
- no-connect marks 17 -> 14
Other:
- note added: "Buzzer"
- note added: "INPUT BOARD ESP v0.7"
- note removed: "Clock RTC"
- note removed: "INPUT BOARD ESP v0.6.3"
- note removed: "Logic Converter"
- moved on the sheet: BZ1, C30, C40, C7, C8, D1, D15, D16, D2, D23, D24, D38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
